File: pcb/dwatum/dwatum.sch (KiCad schematic (older format))
At the start: 33 parts

Commit message: done with schematics from what I can tell
Parts:
- added C? (x2): 10uF, symbol C
- added C? (x2): 1uF, symbol C
- added L?: 2.2uH, symbol INDUCTOR
- added P?: CONN_01X02, symbol CONN_01X02
- added R? (x2): 10K, symbol R
- added U?: TPS62740, symbol TPS62740
- added U?: TPS727xx, symbol TPS727xx
Connections:
- net labels added: +BATT, DW_CE, DW_IRQ, DW_PWR_EN, DW_RSTn, DW_WAKEUP, VAA
- wire segments 121 -> 179
Other:
- moved on the sheet: C?, R?, U?

Commit message: starting on layout
Parts:
- removed C?: 10nF, symbol C
- removed R? (x2): 10K, symbol R
- removed U?: RV-3049-C3, symbol RV-3049-C3
- removed U?: TPS62740, symbol TPS62740
- removed Y?: Crystal, symbol Crystal
- added U4: TPS62740, polypoint:R-PWSON-12, symbol TPS62740
- added X1: CRYSTAL_SMD_4, polypoint:FA-128, symbol CRYSTAL_SMD_4
- A1: renamed from A?; footprint (none) -> polypoint:FRACTUS-2.4GHZ-FR05-S1-N-0-102
- B1: renamed from B?; footprint (none) -> polypoint:2450BM
- C1, C10, C11, C12, C13, C14, C15, C16, C17, C2, C20, C3, C4, C5, C6, C7, C8, C9: renamed from C?; footprint (none) -> Capacitors_SMD:C_0402
- C18, C19: renamed from C?; footprint (none) -> Capacitors_SMD:C_0603
- D1: renamed from D?; footprint (none) -> polypoint:1mm_SQ_4PAD
- J1: renamed from J?; footprint (none) -> polypoint:TC2030
- L1: renamed from L?; footprint (none) -> polypoint:MIPSZ201D
- P1: renamed from P?; footprint (none) -> Pin_Headers:Pin_Header_Straight_1x02
- R1, R2, R3, R4, R5, R6, R7: renamed from R?; footprint (none) -> Resistors_SMD:R_0402
- U1: renamed from U?; footprint (none) -> polypoint:DWM1000_REVERSE
- U2: renamed from U?; footprint (none) -> polypoint:QFN-56-1EP_8x8mm_Pitch0.5mm
- U3: renamed from U?; footprint (none) -> polypoint:WSON-8_1.5x1.5mm
- Y1: renamed from Y?; footprint (none) -> polypoint:ABS05
Connections:
- net labels removed: RTC_CE, ~RTC_INT
- wire segments 179 -> 164

Commit message: working on pcb placement
Parts:
- U1: footprint polypoint:DWM1000_REVERSE -> polypoint:DWM1000_REVERSE_SMD
Connections:
- net labels removed: +3.3V
Changed lines of the file:
@@
 	4100 1550 4000 1550
 Connection ~ 4000 1550
-$Comp
-L +3.3V #PWR03
-U 1 1 553D83E2
-P 3100 1800
-F 0 "#PWR03" H 3100 1650 50  0001 C CNN
-F 1 "+3.3V" H 3100 1940 50  0000 C CNN
-F 2 "" H 3100 1800 60  0000 C CNN
-F 3 "" H 3100 1800 60  0000 C CNN
-	1    3100 1800
-	1    0    0    -1
-$EndComp
 Wire Wire Line
 	3100 1800 3100 2150
@@
 $EndComp
 $Comp
-L GND #PWR04
+L GND #PWR03
 U 1 1 553D8752
 P 2950 5550
-F 0 "#PWR04" H 2950 5300 50  0001 C CNN
+F 0 "#PWR03" H 2950 5300 50  0001 C CNN
 F 1 "GND" H 2950 5400 50  0000 C CNN
 F 2 "" H 2950 5550 60  0000 C CNN
@@
 $EndComp
 $Comp
-L GND #PWR05
+L GND #PWR04
 U 1 1 553D8BE4
 P 5450 3300
-F 0 "#PWR05" H 5450 3050 50  0001 C CNN
+F 0 "#PWR04" H 5450 3050 50  0001 C CNN
 F 1 "GND" H 5450 3150 50  0000 C CNN
 F 2 "" H 5450 3300 60  0000 C CNN
@@
 $EndComp
 $Comp
-L GND #PWR06
+L GND #PWR05
 U 1 1 553D8C16
 P 5450 3800
-F 0 "#PWR06" H 5450 3550 50  0001 C CNN
+F 0 "#PWR05" H 5450 3550 50  0001 C CNN
 F 1 "GND" H 5450 3650 50  0000 C CNN
 F 2 "" H 5450 3800 60  0000 C CNN
@@
 $EndComp
 $Comp
-L GND #PWR07
+L GND #PWR06
 U 1 1 553D8C95
 P 4350 3300
-F 0 "#PWR07" H 4350 3050 50  0001 C CNN
+F 0 "#PWR06" H 4350 3050 50  0001 C CNN
 F 1 "GND" H 4350 3150 50  0000 C CNN
 F 2 "" H 4350 3300 60  0000 C CNN
@@
 $EndComp
 $Comp
-L GND #PWR08
+L GND #PWR07
 U 1 1 553D8CEA
 P 4350 3800
-F 0 "#PWR08" H 4350 3550 50  0001 C CNN
+F 0 "#PWR07" H 4350 3550 50  0001 C CNN
 F 1 "GND" H 4350 3650 50  0000 C CNN
 F 2 "" H 4350 3800 60  0000 C CNN
@@
 Connection ~ 5100 4800
 $Comp
-L GND #PWR09
+L GND #PWR08
 U 1 1 553D92FD
 P 5250 5200
-F 0 "#PWR09" H 5250 4950 50  0001 C CNN
+F 0 "#PWR08" H 5250 4950 50  0001 C CNN
 F 1 "GND" H 5250 5050 50  0000 C CNN
 F 2 "" H 5250 5200 60  0000 C CNN
@@
 $EndComp
 $Comp
-L GND #PWR010
+L GND #PWR09
 U 1 1 553D96A7
 P 4050 5550
-F 0 "#PWR010" H 4050 5300 50  0001 C CNN
+F 0 "#PWR09" H 4050 5300 50  0001 C CNN
 F 1 "GND" H 4050 5400 50  0000 C CNN
 F 2 "" H 4050 5550 60  0000 C CNN
@@
 $EndComp
 $Comp
-L GND #PWR011
+L GND #PWR010
 U 1 1 553D96DC
 P 4900 5550
-F 0 "#PWR011" H 4900 5300 50  0001 C CNN
+F 0 "#PWR010" H 4900 5300 50  0001 C CNN
 F 1 "GND" H 4900 5400 50  0000 C CNN
 F 2 "" H 4900 5550 60  0000 C CNN
@@
 	1700 7300 1500 7300
 $Comp
-L VCC #PWR012
+L VCC #PWR011
 U 1 1 553DCECD
 P 1000 7000
-F 0 "#PWR012" H 1000 6850 50  0001 C CNN
+F 0 "#PWR011" H 1000 6850 50  0001 C CNN
 F 1 "VCC" H 1000 7150 50  0000 C CNN
 F 2 "" H 1000 7000 60  0000 C CNN
@@
 Text GLabel 4150 2850 2    60   Input ~ 0
 LED_RED
+Text GLabel 4150 3050 2    60   Input ~ 0
+LED_BLUE
 Text GLabel 4150 2950 2    60   Input ~ 0
-LED_BLUE
-Text GLabel 4150 3050 2    60   Input ~ 0
 LED_GREEN
 Wire Wire Line
@@
 	5850 3650 5850 3600
 $Comp
-L GND #PWR013
+L GND #PWR012
 U 1 1 553DDE11
 P 6000 3850
-F 0 "#PWR013" H 6000 3600 50  0001 C CNN
+F 0 "#PWR012" H 6000 3600 50  0001 C CNN
 F 1 "GND" H 6000 3700 50  0000 C CNN
 F 2 "" H 6000 3850 60  0000 C CNN
@@
 $EndComp
 $Comp
-L GND #PWR014
+L GND #PWR013
 U 1 1 553DDE9E
 P 7050 3850
-F 0 "#PWR014" H 7050 3600 50  0001 C CNN
+F 0 "#PWR013" H 7050 3600 50  0001 C CNN
 F 1 "GND" H 7050 3700 50  0000 C CNN
 F 2 "" H 7050 3850 60  0000 C CNN
@@
 F 0 "U1" H 8200 2050 60  0000 C CNN
 F 1 "DWM1000" H 9450 2050 60  0000 C CNN
-F 2 "polypoint:DWM1000_REVERSE" H 8600 1600 60  0001 C CNN
+F 2 "polypoint:DWM1000_REVERSE_SMD" H 8600 1600 60  0001 C CNN
 F 3 "" H 8600 1600 60  0000 C CNN
 	1    8600 1600
@@
 BOOTLOADER_TX
 $Comp
-L VCC #PWR015
+L VCC #PWR014
 U 1 1 553DEB0F
 P 3300 6750
-F 0 "#PWR015" H 3300 6600 50  0001 C CNN
+F 0 "#PWR014" H 3300 6600 50  0001 C CNN
 F 1 "VCC" H 3300 6900 50  0000 C CNN
 F 2 "" H 3300 6750 60  0000 C CNN
@@
 $EndComp
 $Comp
-L GND #PWR016
+L GND #PWR015
 U 1 1 553DEB41
 P 3300 7250
-F 0 "#PWR016" H 3300 7000 50  0001 C CNN
+F 0 "#PWR015" H 3300 7000 50  0001 C CNN
 F 1 "GND" H 3300 7100 50  0000 C CNN
 F 2 "" H 3300 7250 60  0000 C CNN
@@
 	4350 7150 4450 7150
 $Comp
-L GND #PWR017
+L GND #PWR016
 U 1 1 553E7E45
 P 10000 1300
-F 0 "#PWR017" H 10000 1050 50  0001 C CNN
+F 0 "#PWR016" H 10000 1050 50  0001 C CNN
 F 1 "GND" H 10000 1150 50  0000 C CNN
 F 2 "" H 10000 1300 60  0000 C CNN
@@
 $EndComp
 $Comp
-L GND #PWR018
+L GND #PWR017
 U 1 1 553E7EF5
 P 10600 1500
-F 0 "#PWR018" H 10600 1250 50  0001 C CNN
+F 0 "#PWR017" H 10600 1250 50  0001 C CNN
 F 1 "GND" H 10600 1350 50  0000 C CNN
 F 2 "" H 10600 1500 60  0000 C CNN
@@
 $EndComp
 $Comp
-L GND #PWR019
+L GND #PWR018
 U 1 1 553E7F42
 P 7850 1950
-F 0 "#PWR019" H 7850 1700 50  0001 C CNN
+F 0 "#PWR018" H 7850 1700 50  0001 C CNN
 F 1 "GND" H 7850 1800 50  0000 C CNN
 F 2 "" H 7850 1950 60  0000 C CNN
@@
 $EndComp
 $Comp
-L GND #PWR020
+L GND #PWR019
 U 1 1 553E7F8F
 P 9300 2450
-F 0 "#PWR020" H 9300 2200 50  0001 C CNN
+F 0 "#PWR019" H 9300 2200 50  0001 C CNN
 F 1 "GND" H 9300 2300 50  0000 C CNN
 F 2 "" H 9300 2450 60  0000 C CNN
@@
 Connection ~ 10000 1300
 $Comp
-L VCC #PWR021
+L VCC #PWR020
 U 1 1 553E8962
 P 7850 1750
-F 0 "#PWR021" H 7850 1600 50  0001 C CNN
+F 0 "#PWR020" H 7850 1600 50  0001 C CNN
 F 1 "VCC" H 7850 1900 50  0000 C CNN
 F 2 "" H 7850 1750 60  0000 C CNN
@@
 	2000 4550 1850 4550
 $Comp
-L GND #PWR022
+L GND #PWR021
 U 1 1 553E9692
 P 9650 5500
-F 0 "#PWR022" H 9650 5250 50  0001 C CNN
+F 0 "#PWR021" H 9650 5250 50  0001 C CNN
 F 1 "GND" H 9650 5350 50  0000 C CNN
 F 2 "" H 9650 5500 60  0000 C CNN
@@
 $EndComp
 $Comp
-L GND #PWR023
+L GND #PWR022
 U 1 1 553E96E1
 P 8450 5650
-F 0 "#PWR023" H 8450 5400 50  0001 C CNN
+F 0 "#PWR022" H 8450 5400 50  0001 C CNN
 F 1 "GND" H 8450 5500 50  0000 C CNN
 F 2 "" H 8450 5650 60  0000 C CNN
@@
 Connection ~ 10200 4750
 $Comp
-L VCC #PWR024
+L VCC #PWR023
 U 1 1 553EA47E
 P 10200 4650
-F 0 "#PWR024" H 10200 4500 50  0001 C CNN
+F 0 "#PWR023" H 10200 4500 50  0001 C CNN
 F 1 "VCC" H 10200 4800 50  0000 C CNN
 F 2 "" H 10200 4650 60  0000 C CNN
@@
 Connection ~ 8300 5100
 $Comp
-L +BATT #PWR025
+L +BATT #PWR024
 U 1 1 553EB11D
 P 7850 4650
-F 0 "#PWR025" H 7850 4500 50  0001 C CNN
+F 0 "#PWR024" H 7850 4500 50  0001 C CNN
 F 1 "+BATT" H 7850 4790 50  0000 C CNN
 F 2 "" H 7850 4650 60  0000 C CNN
@@
 $EndComp
 $Comp
-L +BATT #PWR026
+L +BATT #PWR025
 U 1 1 553ECF03
 P 7750 3700
-F 0 "#PWR026" H 7750 3550 50  0001 C CNN
+F 0 "#PWR025" H 7750 3550 50  0001 C CNN
 F 1 "+BATT" H 7750 3840 50  0000 C CNN
 F 2 "" H 7750 3700 60  0000 C CNN
@@
 $EndComp
 $Comp
-L GND #PWR027
+L GND #PWR026
 U 1 1 553ED2C2
 P 7750 4150
-F 0 "#PWR027" H 7750 3900 50  0001 C CNN
+F 0 "#PWR026" H 7750 3900 50  0001 C CNN
 F 1 "GND" H 7750 4000 50  0000 C CNN
 F 2 "" H 7750 4150 60  0000 C CNN
@@
 $EndComp
 $Comp
-L GND #PWR028
+L GND #PWR027
 U 1 1 553ED31F
 P 9600 4150
-F 0 "#PWR028" H 9600 3900 50  0001 C CNN
+F 0 "#PWR027" H 9600 3900 50  0001 C CNN
 F 1 "GND" H 9600 4000 50  0000 C CNN
 F 2 "" H 9600 4150 60  0000 C CNN
@@
 DW_PWR_EN
 $Comp
-L VAA #PWR029
+L VAA #PWR028
 U 1 1 553EE470
 P 9600 3700
-F 0 "#PWR029" H 9600 3550 50  0001 C CNN
+F 0 "#PWR028" H 9600 3550 50  0001 C CNN
 F 1 "VAA" H 9600 3850 50  0000 C CNN
 F 2 "" H 9600 3700 60  0000 C CNN
@@
 $EndComp
 $Comp
-L GND #PWR030
+L GND #PWR029
 U 1 1 553EF3D8
 P 8550 4400
-F 0 "#PWR030" H 8550 4150 50  0001 C CNN
+F 0 "#PWR029" H 8550 4150 50  0001 C CNN
 F 1 "GND" H 8550 4250 50  0000 C CNN
 F 2 "" H 8550 4400 60  0000 C CNN
@@
 	4700 3650 4700 3800
 $Comp
-L GND #PWR031
+L GND #PWR030
 U 1 1 553F0054
 P 4900 3900
-F 0 "#PWR031" H 4900 3650 50  0001 C CNN
+F 0 "#PWR030" H 4900 3650 50  0001 C CNN
 F 1 "GND" H 4900 3750 50  0000 C CNN
 F 2 "" H 4900 3900 60  0000 C CNN
@@
 $EndComp
 $Comp
-L GND #PWR032
+L GND #PWR031
 U 1 1 553F00AD
 P 4900 3700
-F 0 "#PWR032" H 4900 3450 50  0001 C CNN
+F 0 "#PWR031" H 4900 3450 50  0001 C CNN
 F 1 "GND" H 4900 3550 50  0000 C CNN
 F 2 "" H 4900 3700 60  0000 C CNN
@@
 	-1   0    0    1
 $EndComp
+$Comp
+L VCC #PWR032
+U 1 1 553F9917
+P 3100 1800
+F 0 "#PWR032" H 3100 1650 50  0001 C CNN
+F 1 "VCC" H 3100 1950 50  0000 C CNN
+F 2 "" H 3100 1800 60  0000 C CNN
+F 3 "" H 3100 1800 60  0000 C CNN
+	1    3100 1800
+	1    0    0    -1
+$EndComp
 $EndSCHEMATC

Commit message: most of the routing is done with dwatum
Changed lines of the file:
@@
 	7100 3550 7100 3400
-Wire Wire Line
-	6950 3700 7050 3700
-Wire Wire Line
-	7050 3700 7050 3850
-Wire Wire Line
-	6950 3800 7050 3800
-Connection ~ 7050 3800
 Wire Wire Line
 	6050 3800 6000 3800
@@
 	10000 1250 10000 1350
 Connection ~ 10000 1300
-$Comp
-L VCC #PWR020
-U 1 1 553E8962
-P 7850 1750
-F 0 "#PWR020" H 7850 1600 50  0001 C CNN
-F 1 "VCC" H 7850 1900 50  0000 C CNN
-F 2 "" H 7850 1750 60  0000 C CNN
-F 3 "" H 7850 1750 60  0000 C CNN
-	1    7850 1750
-	0    -1   -1   0
-$EndComp
 Wire Wire Line
 	7950 1750 7850 1750
@@
 	2000 4550 1850 4550
 $Comp
-L GND #PWR021
+L GND #PWR020
 U 1 1 553E9692
 P 9650 5500
-F 0 "#PWR021" H 9650 5250 50  0001 C CNN
+F 0 "#PWR020" H 9650 5250 50  0001 C CNN
 F 1 "GND" H 9650 5350 50  0000 C CNN
 F 2 "" H 9650 5500 60  0000 C CNN
@@
 $EndComp
 $Comp
-L GND #PWR022
+L GND #PWR021
 U 1 1 553E96E1
 P 8450 5650
-F 0 "#PWR022" H 8450 5400 50  0001 C CNN
+F 0 "#PWR021" H 8450 5400 50  0001 C CNN
 F 1 "GND" H 8450 5500 50  0000 C CNN
 F 2 "" H 8450 5650 60  0000 C CNN
@@
 Connection ~ 10200 4750
 $Comp
-L VCC #PWR023
+L VCC #PWR022
 U 1 1 553EA47E
 P 10200 4650
-F 0 "#PWR023" H 10200 4500 50  0001 C CNN
+F 0 "#PWR022" H 10200 4500 50  0001 C CNN
 F 1 "VCC" H 10200 4800 50  0000 C CNN
 F 2 "" H 10200 4650 60  0000 C CNN
@@
 Connection ~ 8300 5100
 $Comp
-L +BATT #PWR024
+L +BATT #PWR023
 U 1 1 553EB11D
 P 7850 4650
-F 0 "#PWR024" H 7850 4500 50  0001 C CNN
+F 0 "#PWR023" H 7850 4500 50  0001 C CNN
 F 1 "+BATT" H 7850 4790 50  0000 C CNN
 F 2 "" H 7850 4650 60  0000 C CNN
@@
 $EndComp
 $Comp
-L +BATT #PWR025
+L +BATT #PWR024
 U 1 1 553ECF03
 P 7750 3700
-F 0 "#PWR025" H 7750 3550 50  0001 C CNN
+F 0 "#PWR024" H 7750 3550 50  0001 C CNN
 F 1 "+BATT" H 7750 3840 50  0000 C CNN
 F 2 "" H 7750 3700 60  0000 C CNN
@@
 $EndComp
 $Comp
-L GND #PWR026
+L GND #PWR025
 U 1 1 553ED2C2
 P 7750 4150
-F 0 "#PWR026" H 7750 3900 50  0001 C CNN
+F 0 "#PWR025" H 7750 3900 50  0001 C CNN
 F 1 "GND" H 7750 4000 50  0000 C CNN
 F 2 "" H 7750 4150 60  0000 C CNN
@@
 $EndComp
 $Comp
-L GND #PWR027
+L GND #PWR026
 U 1 1 553ED31F
 P 9600 4150
-F 0 "#PWR027" H 9600 3900 50  0001 C CNN
+F 0 "#PWR026" H 9600 3900 50  0001 C CNN
 F 1 "GND" H 9600 4000 50  0000 C CNN
 F 2 "" H 9600 4150 60  0000 C CNN
@@
 DW_PWR_EN
 $Comp
-L VAA #PWR028
+L VAA #PWR027
 U 1 1 553EE470
 P 9600 3700
-F 0 "#PWR028" H 9600 3550 50  0001 C CNN
+F 0 "#PWR027" H 9600 3550 50  0001 C CNN
 F 1 "VAA" H 9600 3850 50  0000 C CNN
 F 2 "" H 9600 3700 60  0000 C CNN
@@
 $EndComp
 $Comp
-L GND #PWR029
+L GND #PWR028
 U 1 1 553EF3D8
 P 8550 4400
-F 0 "#PWR029" H 8550 4150 50  0001 C CNN
+F 0 "#PWR028" H 8550 4150 50  0001 C CNN
 F 1 "GND" H 8550 4250 50  0000 C CNN
 F 2 "" H 8550 4400 60  0000 C CNN
@@
 	4700 3650 4700 3800
 $Comp
-L GND #PWR030
+L GND #PWR029
 U 1 1 553F0054
 P 4900 3900
-F 0 "#PWR030" H 4900 3650 50  0001 C CNN
+F 0 "#PWR029" H 4900 3650 50  0001 C CNN
 F 1 "GND" H 4900 3750 50  0000 C CNN
 F 2 "" H 4900 3900 60  0000 C CNN
@@
 $EndComp
 $Comp
-L GND #PWR031
+L GND #PWR030
 U 1 1 553F00AD
 P 4900 3700
-F 0 "#PWR031" H 4900 3450 50  0001 C CNN
+F 0 "#PWR030" H 4900 3450 50  0001 C CNN
 F 1 "GND" H 4900 3550 50  0000 C CNN
 F 2 "" H 4900 3700 60  0000 C CNN
@@
 $EndComp
 $Comp
-L VCC #PWR032
+L VCC #PWR031
 U 1 1 553F9917
 P 3100 1800
-F 0 "#PWR032" H 3100 1650 50  0001 C CNN
+F 0 "#PWR031" H 3100 1650 50  0001 C CNN
 F 1 "VCC" H 3100 1950 50  0000 C CNN
 F 2 "" H 3100 1800 60  0000 C CNN
@@
 	1    0    0    -1
 $EndComp
+$Comp
+L VAA #PWR032
+U 1 1 553FB03D
+P 7850 1750
+F 0 "#PWR032" H 7850 1600 50  0001 C CNN
+F 1 "VAA" H 7850 1900 50  0000 C CNN
+F 2 "" H 7850 1750 60  0000 C CNN
+F 3 "" H 7850 1750 60  0000 C CNN
+	1    7850 1750
+	0    -1   -1   0
+$EndComp
+Connection ~ 7050 3800
+Wire Wire Line
+	6950 3800 7050 3800
+Wire Wire Line
+	7050 3700 7050 3850
+Wire Wire Line
+	6950 3700 7050 3700
 $EndSCHEMATC

Commit message: adding atum footprint and starting from scratch with dwatum adapter board
Parts:
- removed A1: ANT, polypoint:FRACTUS-2.4GHZ-FR05-S1-N-0-102, symbol ANT
- removed B1: 2450BM15A0002, polypoint:2450BM, symbol 2450BM15A0002
- removed C1, C16, C17: 1uF, Capacitors_SMD:C_0402, symbol C
- removed C10, C11: 22pF, Capacitors_SMD:C_0402, symbol C
- removed C12, C13: 12pF, Capacitors_SMD:C_0402, symbol C
- removed C2, C3, C4, C5, C6, C8, C9: 0.1uF, Capacitors_SMD:C_0402, symbol C
- removed C20: 1nF, Capacitors_SMD:C_0402, symbol C
- removed C7: 220pF, Capacitors_SMD:C_0402, symbol C
- removed D1: Led_RGB_CA, polypoint:1mm_SQ_4PAD, symbol Led_RGB_CA
- removed R3: 2.2K, Resistors_SMD:R_0402, symbol R
- removed R4: 56K, Resistors_SMD:R_0402, symbol R
- removed R5, R6, R7: 1K, Resistors_SMD:R_0402, symbol R
- removed U2: CC2538, polypoint:QFN-56-1EP_8x8mm_Pitch0.5mm, symbol CC2538
- removed X1: CRYSTAL_SMD_4, polypoint:FA-128, symbol CRYSTAL_SMD_4
- removed Y1: Crystal, polypoint:ABS05, symbol Crystal
- added U2: ATUM, polypoint:ATUM_SMD, symbol ATUM
Connections:
- net labels removed: LED_BLUE, LED_GREEN, LED_RED
- wire segments 164 -> 73
Other:
- moved on the sheet: J1
