File: pcb/star/rev_a/star.sch (EAGLE design)
At the start: 3 parts

Commit message: got a shape
Parts:
- added A4: FRACTUS-2.4GHZ-FR05-S1-N-0-102, chips:FRACTUS-2.4GHZ-FR05-S1-N-0-102
- added B1: BAL-NRF01D3, chips:BAL-NRF01D3
- added C1: 0.8pF, passives:CAPACITOR
- added C10: 47nF, passives:CAPACITOR
- added C11, C15, C4: 0.1uF, passives:CAPACITOR
- added C13, C18: 1uF, passives:CAPACITOR
- added C14: 4.7uF, passives:CAPACITOR
- added C17: 0.47uF, passives:CAPACITOR
- added C2, C3: 12pF, passives:CAPACITOR
- added C6: 1nF, passives:CAPACITOR
- added C7: 100nF, passives:CAPACITOR
- added C8: 2.2nF, passives:CAPACITOR
- added J1: MICRO_USB_B_HIROSE_ZX62R-B-5P, connector:MICRO_USB_B_HIROSE_ZX62R-B-5P
- added J2: TC2030-JLINK-NL, connector:TC2030-JLINK-NL
- added L1: 15nH, passives:INDUCTOR0402
- added L3: 10uH, passives:INDUCTOR0603
- added LOGO1: UMICH_SOLID_SMALL, logos:UMICH_SOLID_SMALL
- added R10: 25.5k, passives:RESISTOR0402_RES
- added R12: 1M, passives:RESISTOR0402_RES
- added R13: 2M, passives:RESISTOR0402_RES
- added R14: 2.2M, passives:RESISTOR0402_RES
- added R15: 10M, passives:RESISTOR0402_RES
- added R6: 12k, passives:RESISTOR0402_RES
- added U$1, U$2: BAT_FLAT_PAD, connector:BAT_FLAT_PAD
- added U2: LTC4065, chips:LTC4065
- added U4: TPS715AXX, chips:TPS715AXX
- added U5: NRF51822QF, chips:NRF51822QF
- added X1: EPSON-FA-128, crystals:EPSON-FA-128
Connections:
- new net !CHRG: R12.1, R13.2, U2.!CHRG
- new net !FRAM_CS: U5.P15
- new net !FRAM_HOLD: U5.P14
- new net !FRAM_WP: U5.P16
- new net !RTC_INT: U5.P25
- new net AIN3: U5.P02/AIN3
- new net AIN4: U5.P03/AIN4
- new net AIN5: U5.P04/AIN5
- new net AIN6: U5.P05/AIN6
- new net AIN7: U5.P06/AIN7/AREF1
- new net ANTENNA: A4.ANTENNA, B1.SE, C1.1
- new net AVDD: C13.1, C6.1, L1.1, U5.AVDD
- new net BATIN: C15.2, R14.2, R15.1
- new net BOOTLOADER_CTRL: U5.P13
- new net BOOTLOADER_RX: U5.P11
- new net BOOTLOADER_TX: U5.P12
- new net DCC: L3.2, U5.DCC
- new net GND: B1.GND, C1.2, C10.2, C11.2, C13.2, C14.2, C15.1, C17.2, C18.2, C2.2, C3.2, C4.2, C6.2, C7.2, C8.2, J1.GND, J2.GND, R10.1, R13.1, R14.1, R6.1, U$1.-, U$2.-, U2.!EN, U2.GND, U4.GND, U5.GND, X1.GND
- new net I2C_SCL: U5.P01/AIN2
- new net I2C_SDA: U5.P07
- new net LED_BLUE: U5.P19
- new net LED_GREEN: U5.P20
- new net LED_RED: U5.P18
- new net N$10: C2.1, U5.XC2, X1.2
- new net N$13: R10.2, U2.PROG
- new net N$15: C10.1, U5.DEC2
- new net N$17: C7.1, U5.DEC1
- new net N$18: B1.ANT1, U5.ANT1
- new net N$19: B1.ANT2, U5.ANT2
- new net N$20: B1.VDD_PA, C8.1, U5.VDD_PA
- new net N$37: L1.2, L3.1
- new net N$9: C3.1, U5.XC1, X1.1
- new net P08: U5.P08
- new net P09: U5.P09
- new net P10: U5.P10
- new net P17: U5.P17
- new net P21: U5.P21
- new net P22: U5.P22
- new net P23: U5.P23
- new net P24: U5.P24
- new net RTC_CE: U5.P28
- new net SPI_MISO: U5.P29
- new net SPI_MOSI: U5.P30
- new net SPI_SCK: U5.P00/AREF0
- new net SWDCLK: J2.SWDCLK, R6.2, U5.SWDCLK
- new net SWDIO/!RESET: J2.SWDIO, U5.SWDIO/!RESET
- new net VBAT: C4.1, R15.2, U$1.+, U$2.+, U2.BAT, U4.IN
- new net VCC: C11.1, C14.1, C17.1, J2.VCC, U4.OUT, U5.VDD
- new net VUSB: C18.1, J1.+5V, R12.2, U2.VCC

Commit message: new shape
Parts:
- added R1, R2: 10k, passives:RESISTOR0402_RES
Connections:
- net !RTC_INT renamed DW_INT
- removed net !FRAM_CS: U5.P15
- removed net !FRAM_HOLD: U5.P14
- removed net !FRAM_WP: U5.P16
- removed net AIN3: U5.P02/AIN3
- removed net AIN4: U5.P03/AIN4
- removed net AIN5: U5.P04/AIN5
- removed net AIN6: U5.P05/AIN6
- removed net AIN7: U5.P06/AIN7/AREF1
- removed net BOOTLOADER_CTRL: U5.P13
- removed net BOOTLOADER_RX: U5.P11
- removed net BOOTLOADER_TX: U5.P12
- removed net LED_BLUE: U5.P19
- removed net LED_GREEN: U5.P20
- removed net LED_RED: U5.P18
- removed net P08: U5.P08
- removed net P09: U5.P09
- removed net P10: U5.P10
- removed net P17: U5.P17
- removed net P21: U5.P21
- removed net P22: U5.P22
- removed net P23: U5.P23
- removed net P24: U5.P24
- removed net RTC_CE: U5.P28
- removed net SPI_MISO: U5.P29
- removed net SPI_MOSI: U5.P30
- removed net SPI_SCK: U5.P00/AREF0
- net I2C_SCL: now also R2.1, U5.P28; no longer U5.P01/AIN2
- net I2C_SDA: now also R1.1, U5.P29; no longer U5.P07
- net VCC: now also R1.2, R2.2
Changed lines of the file:
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@@
 <part name="GND5" library="supply1" deviceset="GND" device=""/>
 <part name="LOGO1" library="logos" deviceset="UMICH_SOLID" device="_SMALL"/>
+<part name="R1" library="passives" deviceset="RESISTOR" device="0402_RES" value="10k"/>
+<part name="R2" library="passives" deviceset="RESISTOR" device="0402_RES" value="10k"/>
+<part name="P+2" library="supply1" deviceset="VCC" device=""/>
 </parts>
 <sheets>
@@
 <instance part="GND5" gate="1" x="172.72" y="137.16"/>
 <instance part="LOGO1" gate="G$1" x="200.66" y="114.3"/>
+<instance part="R1" gate="G$1" x="137.16" y="127" rot="R90"/>
+<instance part="R2" gate="G$1" x="144.78" y="127" rot="R90"/>
+<instance part="P+2" gate="VCC" x="139.7" y="139.7"/>
 </instances>
 <busses>
@@
 <wire x1="172.72" y1="152.4" x2="172.72" y2="154.94" width="0.1524" layer="91"/>
 </segment>
+<segment>
+<pinref part="R1" gate="G$1" pin="2"/>
+<wire x1="137.16" y1="132.08" x2="137.16" y2="134.62" width="0.1524" layer="91"/>
+<pinref part="R2" gate="G$1" pin="2"/>
+<wire x1="137.16" y1="134.62" x2="139.7" y2="134.62" width="0.1524" layer="91"/>
+<wire x1="139.7" y1="134.62" x2="144.78" y2="134.62" width="0.1524" layer="91"/>
+<wire x1="144.78" y1="134.62" x2="144.78" y2="132.08" width="0.1524" layer="91"/>
+<pinref part="P+2" gate="VCC" pin="VCC"/>
+<wire x1="139.7" y1="134.62" x2="139.7" y2="137.16" width="0.1524" layer="91"/>
+<junction x="139.7" y="134.62"/>
+</segment>
 </net>
 <net name="N$15" class="0">
@@
 <wire x1="114.3" y1="58.42" x2="114.3" y2="53.34" width="0.1524" layer="91"/>
 <pinref part="U5" gate="G$1" pin="DEC2"/>
-</segment>
-</net>
-<net name="BOOTLOADER_RX" class="0">
-<segment>
-<pinref part="U5" gate="G$1" pin="P11"/>
-<wire x1="60.96" y1="86.36" x2="53.34" y2="86.36" width="0.1524" layer="91"/>
-<label x="53.34" y="86.36" size="1.27" layer="95" rot="R180" xref="yes"/>
 </segment>
 </net>
@@
 </segment>
 </net>
-<net name="!FRAM_CS" class="0">
-<segment>
-<label x="53.34" y="76.2" size="1.27" layer="95" rot="R180" xref="yes"/>
-<pinref part="U5" gate="G$1" pin="P15"/>
-<wire x1="53.34" y1="76.2" x2="60.96" y2="76.2" width="0.1524" layer="91"/>
-</segment>
-</net>
-<net name="!FRAM_HOLD" class="0">
-<segment>
-<label x="53.34" y="78.74" size="1.27" layer="95" rot="R180" xref="yes"/>
-<pinref part="U5" gate="G$1" pin="P14"/>
-<wire x1="53.34" y1="78.74" x2="60.96" y2="78.74" width="0.1524" layer="91"/>
-</segment>
-</net>
-<net name="!FRAM_WP" class="0">
-<segment>
-<label x="111.76" y="121.92" size="1.27" layer="95" xref="yes"/>
-<pinref part="U5" gate="G$1" pin="P16"/>
-<wire x1="111.76" y1="121.92" x2="106.68" y2="121.92" width="0.1524" layer="91"/>
-</segment>
-</net>
-<net name="BOOTLOADER_TX" class="0">
-<segment>
-<pinref part="U5" gate="G$1" pin="P12"/>
-<wire x1="60.96" y1="83.82" x2="53.34" y2="83.82" width="0.1524" layer="91"/>
-<label x="53.34" y="83.82" size="1.27" layer="95" rot="R180" xref="yes"/>
-</segment>
-</net>
-<net name="BOOTLOADER_CTRL" class="0">
-<segment>
-<pinref part="U5" gate="G$1" pin="P13"/>
-<wire x1="60.96" y1="81.28" x2="53.34" y2="81.28" width="0.1524" layer="91"/>
-<label x="53.34" y="81.28" size="1.27" layer="95" rot="R180" xref="yes"/>
-</segment>
-</net>
-<net name="I2C_SDA" class="0">
-<segment>
-<label x="53.34" y="99.06" size="1.27" layer="95" rot="R180" xref="yes"/>
-<pinref part="U5" gate="G$1" pin="P07"/>
-<wire x1="53.34" y1="99.06" x2="60.96" y2="99.06" width="0.1524" layer="91"/>
-</segment>
-</net>
-<net name="SPI_SCK" class="0">
-<segment>
-<label x="53.34" y="116.84" size="1.27" layer="95" rot="R180" xref="yes"/>
-<pinref part="U5" gate="G$1" pin="P00/AREF0"/>
-<wire x1="53.34" y1="116.84" x2="60.96" y2="116.84" width="0.1524" layer="91"/>
-</segment>
-</net>
-<net name="!RTC_INT" class="0">
+<net name="DW_INT" class="0">
 <segment>
 <label x="111.76" y="96.52" size="1.27" layer="95" xref="yes"/>
@@
 </segment>
 </net>
-<net name="LED_BLUE" class="0">
-<segment>
-<label x="111.76" y="114.3" size="1.27" layer="95" xref="yes"/>
-<pinref part="U5" gate="G$1" pin="P19"/>
-<wire x1="111.76" y1="114.3" x2="106.68" y2="114.3" width="0.1524" layer="91"/>
-</segment>
-</net>
-<net name="LED_GREEN" class="0">
-<segment>
-<label x="111.76" y="111.76" size="1.27" layer="95" xref="yes"/>
-<pinref part="U5" gate="G$1" pin="P20"/>
-<wire x1="106.68" y1="111.76" x2="111.76" y2="111.76" width="0.1524" layer="91"/>
-</segment>
-</net>
-<net name="LED_RED" class="0">
-<segment>
-<label x="111.76" y="116.84" size="1.27" layer="95" xref="yes"/>
-<pinref part="U5" gate="G$1" pin="P18"/>
-<wire x1="106.68" y1="116.84" x2="111.76" y2="116.84" width="0.1524" layer="91"/>
-</segment>
-</net>
-<net name="P17" class="0">
-<segment>
-<pinref part="U5" gate="G$1" pin="P17"/>
-<wire x1="106.68" y1="119.38" x2="111.76" y2="119.38" width="0.1524" layer="91"/>
-<label x="111.76" y="119.38" size="1.27" layer="95" xref="yes"/>
-</segment>
-</net>
-<net name="I2C_SCL" class="0">
-<segment>
-<label x="53.34" y="114.3" size="1.27" layer="95" rot="R180" xref="yes"/>
-<pinref part="U5" gate="G$1" pin="P01/AIN2"/>
-<wire x1="53.34" y1="114.3" x2="60.96" y2="114.3" width="0.1524" layer="91"/>
-</segment>
-</net>
-<net name="SPI_MOSI" class="0">
-<segment>
-<label x="111.76" y="83.82" size="1.27" layer="95" xref="yes"/>
-<pinref part="U5" gate="G$1" pin="P30"/>
-<wire x1="106.68" y1="83.82" x2="111.76" y2="83.82" width="0.1524" layer="91"/>
-</segment>
-</net>
-<net name="SPI_MISO" class="0">
+<net name="I2C_SDA" class="0">
 <segment>
 <label x="111.76" y="86.36" size="1.27" layer="95" xref="yes"/>
@@
 <wire x1="111.76" y1="86.36" x2="106.68" y2="86.36" width="0.1524" layer="91"/>
 </segment>
-</net>
-<net name="RTC_CE" class="0">
+<segment>
+<pinref part="R1" gate="G$1" pin="1"/>
+<wire x1="137.16" y1="121.92" x2="137.16" y2="119.38" width="0.1524" layer="91"/>
+<wire x1="137.16" y1="119.38" x2="134.62" y2="119.38" width="0.1524" layer="91"/>
+<label x="134.62" y="119.38" size="1.27" layer="95" rot="R180" xref="yes"/>
+</segment>
+</net>
+<net name="I2C_SCL" class="0">
 <segment>
 <label x="111.76" y="88.9" size="1.27" layer="95" xref="yes"/>
 <pinref part="U5" gate="G$1" pin="P28"/>
 <wire x1="111.76" y1="88.9" x2="106.68" y2="88.9" width="0.1524" layer="91"/>
+</segment>
+<segment>
+<pinref part="R2" gate="G$1" pin="1"/>
+<wire x1="144.78" y1="121.92" x2="144.78" y2="116.84" width="0.1524" layer="91"/>
+<wire x1="144.78" y1="116.84" x2="134.62" y2="116.84" width="0.1524" layer="91"/>
+<label x="134.62" y="116.84" size="1.27" layer="95" rot="R180" xref="yes"/>
 </segment>
 </net>
@@
 </segment>
 </net>
-<net name="AIN3" class="0">
-<segment>
-<label x="53.34" y="111.76" size="1.27" layer="95" rot="R180" xref="yes"/>
-<pinref part="U5" gate="G$1" pin="P02/AIN3"/>
-<wire x1="53.34" y1="111.76" x2="60.96" y2="111.76" width="0.1524" layer="91"/>
-</segment>
-</net>
-<net name="AIN4" class="0">
-<segment>
-<label x="53.34" y="109.22" size="1.27" layer="95" rot="R180" xref="yes"/>
-<pinref part="U5" gate="G$1" pin="P03/AIN4"/>
-<wire x1="53.34" y1="109.22" x2="60.96" y2="109.22" width="0.1524" layer="91"/>
-</segment>
-</net>
-<net name="AIN5" class="0">
-<segment>
-<label x="53.34" y="106.68" size="1.27" layer="95" rot="R180" xref="yes"/>
-<pinref part="U5" gate="G$1" pin="P04/AIN5"/>
-<wire x1="53.34" y1="106.68" x2="60.96" y2="106.68" width="0.1524" layer="91"/>
-</segment>
-</net>
-<net name="AIN6" class="0">
-<segment>
-<label x="53.34" y="104.14" size="1.27" layer="95" rot="R180" xref="yes"/>
-<pinref part="U5" gate="G$1" pin="P05/AIN6"/>
-<wire x1="53.34" y1="104.14" x2="60.96" y2="104.14" width="0.1524" layer="91"/>
-</segment>
-</net>
-<net name="AIN7" class="0">
-<segment>
-<label x="53.34" y="101.6" size="1.27" layer="95" rot="R180" xref="yes"/>
-<pinref part="U5" gate="G$1" pin="P06/AIN7/AREF1"/>
-<wire x1="53.34" y1="101.6" x2="60.96" y2="101.6" width="0.1524" layer="91"/>
-</segment>
-</net>
-<net name="P10" class="0">
-<segment>
-<pinref part="U5" gate="G$1" pin="P10"/>
-<wire x1="60.96" y1="88.9" x2="53.34" y2="88.9" width="0.1524" layer="91"/>
-<label x="53.34" y="88.9" size="1.27" layer="95" rot="R180" xref="yes"/>
-</segment>
-</net>
-<net name="P09" class="0">
-<segment>
-<pinref part="U5" gate="G$1" pin="P09"/>
-<wire x1="60.96" y1="91.44" x2="53.34" y2="91.44" width="0.1524" layer="91"/>
-<label x="53.34" y="91.44" size="1.27" layer="95" rot="R180" xref="yes"/>
-</segment>
-</net>
-<net name="P08" class="0">
-<segment>
-<pinref part="U5" gate="G$1" pin="P08"/>
-<wire x1="60.96" y1="93.98" x2="53.34" y2="93.98" width="0.1524" layer="91"/>
-<label x="53.34" y="93.98" size="1.27" layer="95" rot="R180" xref="yes"/>
-</segment>
-</net>
-<net name="P24" class="0">
-<segment>
-<label x="111.76" y="99.06" size="1.27" layer="95" xref="yes"/>
-<pinref part="U5" gate="G$1" pin="P24"/>
-<wire x1="106.68" y1="99.06" x2="111.76" y2="99.06" width="0.1524" layer="91"/>
-</segment>
-</net>
-<net name="P23" class="0">
-<segment>
-<label x="111.76" y="104.14" size="1.27" layer="95" xref="yes"/>
-<pinref part="U5" gate="G$1" pin="P23"/>
-<wire x1="106.68" y1="104.14" x2="111.76" y2="104.14" width="0.1524" layer="91"/>
-</segment>
-</net>
-<net name="P22" class="0">
-<segment>
-<label x="111.76" y="106.68" size="1.27" layer="95" xref="yes"/>
-<pinref part="U5" gate="G$1" pin="P22"/>
-<wire x1="106.68" y1="106.68" x2="111.76" y2="106.68" width="0.1524" layer="91"/>
-</segment>
-</net>
-<net name="P21" class="0">
-<segment>
-<label x="111.76" y="109.22" size="1.27" layer="95" xref="yes"/>
-<pinref part="U5" gate="G$1" pin="P21"/>
-<wire x1="106.68" y1="109.22" x2="111.76" y2="109.22" width="0.1524" layer="91"/>
-</segment>
-</net>

Commit message: more routing
Parts:
- removed R13: 2M, passives:RESISTOR0402_RES
- added D1, D2: (no value), SparkFun-LED:LED0603
- added R3: 1k, passives:RESISTOR0402_RES
- R10: value 25.5k -> 2k 1%
- R12: value 1M -> 1k
Connections:
- new net !CHRG1: D2.A, R3.1
- new net N$5: D1.C, U2.!CHRG
- new net N$6: D2.C, U5.P24
- net !CHRG: now also D1.A; no longer R13.2, U2.!CHRG
- net GND: no longer R13.1
- net VCC: now also R3.2
Other:
- moved on the sheet: C18, R10
Changed lines of the file:
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@@
 <part name="FRAME2" library="frames" deviceset="LETTER_L" device=""/>
 <part name="U2" library="chips" deviceset="LTC4065" device=""/>
-<part name="R12" library="passives" deviceset="RESISTOR" device="0402_RES" value="1M"/>
+<part name="R12" library="passives" deviceset="RESISTOR" device="0402_RES" value="1k"/>
 <part name="C18" library="passives" deviceset="CAPACITOR" device="" value="1uF"/>
-<part name="R10" library="passives" deviceset="RESISTOR" device="0402_RES" value="25.5k"/>
-<part name="R13" library="passives" deviceset="RESISTOR" device="0402_RES" value="2M"/>
+<part name="R10" library="passives" deviceset="RESISTOR" device="0402_RES" value="2k 1%"/>
 <part name="SUPPLY5" library="supply1" deviceset="GND" device=""/>
 <part name="U4" library="chips" deviceset="TPS715AXX" device=""/>
@@
 <part name="SUPPLY14" library="supply1" deviceset="GND" device=""/>
 <part name="SUPPLY1" library="supply1" deviceset="GND" device=""/>
-<part name="SUPPLY2" library="supply1" deviceset="GND" device=""/>
 <part name="SUPPLY3" library="supply1" deviceset="GND" device=""/>
 <part name="SUPPLY4" library="supply1" deviceset="GND" device=""/>
@@
 <part name="R2" library="passives" deviceset="RESISTOR" device="0402_RES" value="10k"/>
 <part name="P+2" library="supply1" deviceset="VCC" device=""/>
+<part name="D1" library="SparkFun-LED" deviceset="LED" device="0603"/>
+<part name="SUPPLY2" library="supply1" deviceset="GND" device=""/>
+<part name="R3" library="passives" deviceset="RESISTOR" device="0402_RES" value="1k"/>
+<part name="D2" library="SparkFun-LED" deviceset="LED" device="0603"/>
+<part name="P+5" library="supply1" deviceset="VCC" device=""/>
 </parts>
 <sheets>
@@
 <instance part="U2" gate="G$1" x="114.3" y="78.74"/>
 <instance part="R12" gate="G$1" x="91.44" y="86.36" rot="R90"/>
-<instance part="C18" gate="G$1" x="73.66" y="78.74"/>
-<instance part="R10" gate="G$1" x="137.16" y="71.12" rot="R90"/>
-<instance part="R13" gate="G$1" x="91.44" y="71.12" rot="R90"/>
-<instance part="SUPPLY5" gate="1" x="134.62" y="53.34"/>
+<instance part="C18" gate="G$1" x="73.66" y="81.28"/>
+<instance part="R10" gate="G$1" x="139.7" y="71.12" rot="R90"/>
+<instance part="SUPPLY5" gate="1" x="132.08" y="53.34"/>
 <instance part="U4" gate="G$1" x="200.66" y="83.82"/>
 <instance part="SUPPLY6" gate="1" x="200.66" y="68.58"/>
@@
 <instance part="SUPPLY14" gate="1" x="137.16" y="96.52"/>
 <instance part="SUPPLY1" gate="1" x="99.06" y="53.34"/>
-<instance part="SUPPLY2" gate="1" x="91.44" y="53.34"/>
 <instance part="SUPPLY3" gate="1" x="68.58" y="53.34"/>
 <instance part="SUPPLY4" gate="1" x="152.4" y="53.34"/>
 <instance part="SUPPLY7" gate="1" x="160.02" y="53.34"/>
 <instance part="U$2" gate="G$1" x="124.46" y="121.92"/>
+<instance part="D1" gate="G$1" x="91.44" y="76.2"/>
+<instance part="SUPPLY2" gate="1" x="139.7" y="53.34"/>
 </instances>
 <busses>
@@
 <net name="GND" class="0">
 <segment>
-<pinref part="R13" gate="G$1" pin="1"/>
-<pinref part="SUPPLY2" gate="1" pin="GND"/>
-<wire x1="91.44" y1="55.88" x2="91.44" y2="66.04" width="0.1524" layer="91"/>
-</segment>
-<segment>
 <pinref part="U2" gate="G$1" pin="!EN"/>
 <wire x1="101.6" y1="71.12" x2="99.06" y2="71.12" width="0.1524" layer="91"/>
@@
 </segment>
 <segment>
-<pinref part="R10" gate="G$1" pin="1"/>
-<wire x1="134.62" y1="55.88" x2="134.62" y2="63.5" width="0.1524" layer="91"/>
 <pinref part="SUPPLY5" gate="1" pin="GND"/>
-<wire x1="134.62" y1="63.5" x2="137.16" y2="63.5" width="0.1524" layer="91"/>
-<wire x1="137.16" y1="63.5" x2="137.16" y2="66.04" width="0.1524" layer="91"/>
-<wire x1="134.62" y1="63.5" x2="132.08" y2="63.5" width="0.1524" layer="91"/>
-<junction x="134.62" y="63.5"/>
-<wire x1="132.08" y1="63.5" x2="132.08" y2="71.12" width="0.1524" layer="91"/>
+<wire x1="132.08" y1="55.88" x2="132.08" y2="71.12" width="0.1524" layer="91"/>
 <pinref part="U2" gate="G$1" pin="GND"/>
 <wire x1="132.08" y1="71.12" x2="129.54" y2="71.12" width="0.1524" layer="91"/>
@@
 <segment>
 <pinref part="C18" gate="G$1" pin="2"/>
-<wire x1="73.66" y1="73.66" x2="73.66" y2="66.04" width="0.1524" layer="91"/>
+<wire x1="73.66" y1="76.2" x2="73.66" y2="66.04" width="0.1524" layer="91"/>
 <wire x1="73.66" y1="66.04" x2="68.58" y2="66.04" width="0.1524" layer="91"/>
 <pinref part="SUPPLY3" gate="1" pin="GND"/>
@@
 <wire x1="160.02" y1="60.96" x2="160.02" y2="55.88" width="0.1524" layer="91"/>
 </segment>
+<segment>
+<pinref part="R10" gate="G$1" pin="1"/>
+<pinref part="SUPPLY2" gate="1" pin="GND"/>
+<wire x1="139.7" y1="55.88" x2="139.7" y2="66.04" width="0.1524" layer="91"/>
+</segment>
 </net>
 <net name="VCC" class="0">
@@
 <segment>
 <pinref part="C18" gate="G$1" pin="1"/>
-<wire x1="73.66" y1="93.98" x2="73.66" y2="81.28" width="0.1524" layer="91"/>
+<wire x1="73.66" y1="93.98" x2="73.66" y2="83.82" width="0.1524" layer="91"/>
 <pinref part="J1" gate="G$1" pin="+5V"/>
 <wire x1="55.88" y1="83.82" x2="60.96" y2="83.82" width="0.1524" layer="91"/>
@@
 <segment>
 <pinref part="R12" gate="G$1" pin="1"/>
-<pinref part="R13" gate="G$1" pin="2"/>
-<wire x1="91.44" y1="76.2" x2="91.44" y2="78.74" width="0.1524" layer="91"/>
-<pinref part="U2" gate="G$1" pin="!CHRG"/>
 <wire x1="91.44" y1="78.74" x2="91.44" y2="81.28" width="0.1524" layer="91"/>
-<wire x1="101.6" y1="78.74" x2="91.44" y2="78.74" width="0.1524" layer="91"/>
-<junction x="91.44" y="78.74"/>
-<wire x1="91.44" y1="78.74" x2="88.9" y2="78.74" width="0.1524" layer="91"/>
-<label x="88.9" y="78.74" size="1.27" layer="95" rot="R180" xref="yes"/>
+<pinref part="D1" gate="G$1" pin="A"/>
 </segment>
 </net>
@@
 <segment>
 <pinref part="R10" gate="G$1" pin="2"/>
-<wire x1="137.16" y1="76.2" x2="137.16" y2="78.74" width="0.1524" layer="91"/>
+<wire x1="139.7" y1="76.2" x2="139.7" y2="78.74" width="0.1524" layer="91"/>
 <pinref part="U2" gate="G$1" pin="PROG"/>
-<wire x1="137.16" y1="78.74" x2="129.54" y2="78.74" width="0.1524" layer="91"/>
+<wire x1="139.7" y1="78.74" x2="129.54" y2="78.74" width="0.1524" layer="91"/>
 </segment>
 </net>
@@
 <wire x1="160.02" y1="71.12" x2="162.56" y2="71.12" width="0.1524" layer="91"/>
 <junction x="160.02" y="71.12"/>
+</segment>
+</net>
+<net name="N$5" class="0">
+<segment>
+<pinref part="D1" gate="G$1" pin="C"/>
+<wire x1="91.44" y1="71.12" x2="91.44" y2="68.58" width="0.1524" layer="91"/>
+<wire x1="91.44" y1="68.58" x2="96.52" y2="68.58" width="0.1524" layer="91"/>
+<wire x1="96.52" y1="68.58" x2="96.52" y2="78.74" width="0.1524" layer="91"/>
+<pinref part="U2" gate="G$1" pin="!CHRG"/>
+<wire x1="96.52" y1="78.74" x2="101.6" y2="78.74" width="0.1524" layer="91"/>
 </segment>
 </net>
@@
 <instance part="R2" gate="G$1" x="144.78" y="127" rot="R90"/>
 <instance part="P+2" gate="VCC" x="139.7" y="139.7"/>
+<instance part="R3" gate="G$1" x="119.38" y="116.84" rot="R90"/>
+<instance part="D2" gate="G$1" x="119.38" y="106.68"/>
+<instance part="P+5" gate="VCC" x="119.38" y="127"/>
 </instances>
 <busses>
@@
 <wire x1="139.7" y1="134.62" x2="139.7" y2="137.16" width="0.1524" layer="91"/>
 <junction x="139.7" y="134.62"/>
+</segment>
+<segment>
+<pinref part="R3" gate="G$1" pin="2"/>
+<wire x1="119.38" y1="121.92" x2="119.38" y2="124.46" width="0.1524" layer="91"/>
+<pinref part="P+5" gate="VCC" pin="VCC"/>
 </segment>
 </net>
@@
 </segment>
 </net>
+<net name="!CHRG1" class="0">
+<segment>
+<pinref part="R3" gate="G$1" pin="1"/>
+<wire x1="119.38" y1="109.22" x2="119.38" y2="111.76" width="0.1524" layer="91"/>
+<pinref part="D2" gate="G$1" pin="A"/>
+</segment>
+</net>
+<net name="N$6" class="0">
+<segment>
+<pinref part="U5" gate="G$1" pin="P24"/>
+<pinref part="D2" gate="G$1" pin="C"/>
+<wire x1="106.68" y1="99.06" x2="119.38" y2="99.06" width="0.1524" layer="91"/>
+<wire x1="119.38" y1="99.06" x2="119.38" y2="101.6" width="0.1524" layer="91"/>
+</segment>
+</net>
