File: pcb/star/rev_a/star.sch (EAGLE design)
At the start: 40 parts, among them J1 MICRO_USB_B_HIROSE_ZX62R-B-5P, J2 TC2030-JLINK-NL, U2 LTC4065, U4 TPS715AXX, U5 NRF51822QF, X1 EPSON-FA-128

Commit message: updating pcb
Parts:
- removed J1: MICRO_USB_B_HIROSE_ZX62R-B-5P, connector:MICRO_USB_B_HIROSE_ZX62R-B-5P
- removed U$1, U$2: BAT_FLAT_PAD, connector:BAT_FLAT_PAD
- added J3: MICRO_USB_B_HIROSE_ZX62-B-5PA(11), connector:MICRO_USB_B_HIROSE_ZX62-B-5PA(11)
- added J4: TC2030-JLINK-NL, connector:TC2030-JLINK-NL
- added U$3, U$4: BAT_HOLE, connector:BAT_HOLE
- added U3: TRIPOINT, tripoint:TRIPOINT
Connections:
- net GND: now also J3.GND, J4.GND, U$3.-, U$4.-; no longer J1.GND, U$1.-, U$2.-
- net VBAT: now also U$3.+, U$4.+; no longer U$1.+, U$2.+
- net VCC: now also J4.VCC
- net VUSB: now also J3.+5V; no longer J1.+5V
Changed lines of the file:
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@@
 <part name="A2" library="chips" deviceset="TAIYO-YUDEN-AH086M" device=""/>
 <part name="A3" library="chips" deviceset="TAIYO-YUDEN-AH086M" device=""/>
-<part name="J1" library="connector" deviceset="MICRO_USB_B_HIROSE_ZX62R-B-5P" device=""/>
 <part name="GND4" library="supply1" deviceset="GND" device=""/>
 <part name="X1" library="crystals" deviceset="EPSON-FA-128" device=""/>
@@
 <part name="C17" library="passives" deviceset="CAPACITOR" device="" value="0.47uF"/>
 <part name="C15" library="passives" deviceset="CAPACITOR" device="" value="0.1uF"/>
-<part name="U$1" library="connector" deviceset="BAT_FLAT_PAD" device=""/>
 <part name="SUPPLY14" library="supply1" deviceset="GND" device=""/>
 <part name="SUPPLY1" library="supply1" deviceset="GND" device=""/>
@@
 <part name="SUPPLY4" library="supply1" deviceset="GND" device=""/>
 <part name="SUPPLY7" library="supply1" deviceset="GND" device=""/>
-<part name="U$2" library="connector" deviceset="BAT_FLAT_PAD" device=""/>
 <part name="J2" library="connector" deviceset="TC2030-JLINK" device="-NL"/>
 <part name="P+4" library="supply1" deviceset="VCC" device=""/>
@@
 <part name="D2" library="SparkFun-LED" deviceset="LED" device="0603"/>
 <part name="P+5" library="supply1" deviceset="VCC" device=""/>
+<part name="J3" library="connector" deviceset="MICRO_USB_B_HIROSE_ZX62-B-5PA(11)" device=""/>
+<part name="FRAME3" library="frames" deviceset="LETTER_L" device=""/>
+<part name="U3" library="tripoint" deviceset="TRIPOINT" device=""/>
+<part name="U$3" library="connector" deviceset="BAT_HOLE" device=""/>
+<part name="U$4" library="connector" deviceset="BAT_HOLE" device=""/>
+<part name="J4" library="connector" deviceset="TC2030-JLINK" device="-NL"/>
+<part name="P+6" library="supply1" deviceset="VCC" device=""/>
+<part name="GND1" library="supply1" deviceset="GND" device=""/>
 </parts>
 <sheets>
@@
 <instance part="FRAME1" gate="G$1" x="0" y="0"/>
 <instance part="FRAME1" gate="G$2" x="147.32" y="0"/>
-<instance part="A1" gate="G$1" x="147.32" y="142.24"/>
-<instance part="A2" gate="G$1" x="162.56" y="142.24"/>
-<instance part="A3" gate="G$1" x="175.26" y="142.24"/>
-<instance part="J1" gate="G$1" x="48.26" y="78.74" rot="MR0"/>
 <instance part="U2" gate="G$1" x="114.3" y="78.74"/>
 <instance part="R12" gate="G$1" x="91.44" y="86.36" rot="R90"/>
@@
 <attribute name="VALUE" x="168.91" y="63.119" size="1.778" layer="96" rot="R180"/>
 </instance>
-<instance part="U$1" gate="G$1" x="124.46" y="106.68"/>
 <instance part="SUPPLY14" gate="1" x="137.16" y="96.52"/>
 <instance part="SUPPLY1" gate="1" x="99.06" y="53.34"/>
@@
 <instance part="SUPPLY4" gate="1" x="152.4" y="53.34"/>
 <instance part="SUPPLY7" gate="1" x="160.02" y="53.34"/>
-<instance part="U$2" gate="G$1" x="124.46" y="121.92"/>
 <instance part="D1" gate="G$1" x="91.44" y="76.2"/>
 <instance part="SUPPLY2" gate="1" x="139.7" y="53.34"/>
+<instance part="J3" gate="G$1" x="48.26" y="78.74" rot="MR0"/>
+<instance part="U$3" gate="G$1" x="124.46" y="134.62"/>
+<instance part="U$4" gate="G$1" x="124.46" y="147.32"/>
 </instances>
 <busses>
@@
 <segment>
 <pinref part="SUPPLY14" gate="1" pin="GND"/>
-<pinref part="U$1" gate="G$1" pin="-"/>
-<wire x1="137.16" y1="99.06" x2="137.16" y2="104.14" width="0.1524" layer="91"/>
-<wire x1="137.16" y1="104.14" x2="134.62" y2="104.14" width="0.1524" layer="91"/>
-<pinref part="U$2" gate="G$1" pin="-"/>
-<wire x1="134.62" y1="119.38" x2="137.16" y2="119.38" width="0.1524" layer="91"/>
-<wire x1="137.16" y1="119.38" x2="137.16" y2="104.14" width="0.1524" layer="91"/>
-<junction x="137.16" y="104.14"/>
+<wire x1="137.16" y1="132.08" x2="137.16" y2="99.06" width="0.1524" layer="91"/>
+<pinref part="U$4" gate="G$1" pin="-"/>
+<wire x1="134.62" y1="144.78" x2="137.16" y2="144.78" width="0.1524" layer="91"/>
+<wire x1="137.16" y1="144.78" x2="137.16" y2="132.08" width="0.1524" layer="91"/>
+<pinref part="U$3" gate="G$1" pin="-"/>
+<wire x1="134.62" y1="132.08" x2="137.16" y2="132.08" width="0.1524" layer="91"/>
+<junction x="137.16" y="132.08"/>
 </segment>
 <segment>
@@
 <pinref part="SUPPLY3" gate="1" pin="GND"/>
 <wire x1="68.58" y1="66.04" x2="68.58" y2="55.88" width="0.1524" layer="91"/>
-<pinref part="J1" gate="G$1" pin="GND"/>
-<wire x1="55.88" y1="73.66" x2="60.96" y2="73.66" width="0.1524" layer="91"/>
 <wire x1="60.96" y1="73.66" x2="60.96" y2="66.04" width="0.1524" layer="91"/>
 <wire x1="60.96" y1="66.04" x2="68.58" y2="66.04" width="0.1524" layer="91"/>
 <junction x="68.58" y="66.04"/>
+<pinref part="J3" gate="G$1" pin="GND"/>
+<wire x1="55.88" y1="73.66" x2="60.96" y2="73.66" width="0.1524" layer="91"/>
 </segment>
 <segment>
@@
 <pinref part="C18" gate="G$1" pin="1"/>
 <wire x1="73.66" y1="93.98" x2="73.66" y2="83.82" width="0.1524" layer="91"/>
-<pinref part="J1" gate="G$1" pin="+5V"/>
-<wire x1="55.88" y1="83.82" x2="60.96" y2="83.82" width="0.1524" layer="91"/>
-<wire x1="60.96" y1="83.82" x2="60.96" y2="93.98" width="0.1524" layer="91"/>
 <wire x1="60.96" y1="93.98" x2="73.66" y2="93.98" width="0.1524" layer="91"/>
 <junction x="73.66" y="93.98"/>
@@
 <wire x1="73.66" y1="93.98" x2="91.44" y2="93.98" width="0.1524" layer="91"/>
 <junction x="91.44" y="93.98"/>
+<wire x1="60.96" y1="93.98" x2="60.96" y2="83.82" width="0.1524" layer="91"/>
+<pinref part="J3" gate="G$1" pin="+5V"/>
+<wire x1="60.96" y1="83.82" x2="55.88" y2="83.82" width="0.1524" layer="91"/>
 </segment>
 </net>
@@
 <net name="VBAT" class="0">
 <segment>
-<pinref part="U$1" gate="G$1" pin="+"/>
 <pinref part="U2" gate="G$1" pin="BAT"/>
 <pinref part="R15" gate="G$1" pin="2"/>
@@
 <junction x="152.4" y="86.36"/>
 <junction x="182.88" y="86.36"/>
-<wire x1="134.62" y1="109.22" x2="152.4" y2="109.22" width="0.1524" layer="91"/>
-<wire x1="152.4" y1="109.22" x2="152.4" y2="86.36" width="0.1524" layer="91"/>
-<pinref part="U$2" gate="G$1" pin="+"/>
-<wire x1="134.62" y1="124.46" x2="152.4" y2="124.46" width="0.1524" layer="91"/>
-<wire x1="152.4" y1="124.46" x2="152.4" y2="109.22" width="0.1524" layer="91"/>
-<junction x="152.4" y="109.22"/>
+<wire x1="152.4" y1="137.16" x2="152.4" y2="86.36" width="0.1524" layer="91"/>
+<pinref part="U$4" gate="G$1" pin="+"/>
+<wire x1="152.4" y1="137.16" x2="152.4" y2="149.86" width="0.1524" layer="91"/>
+<wire x1="152.4" y1="149.86" x2="134.62" y2="149.86" width="0.1524" layer="91"/>
+<pinref part="U$3" gate="G$1" pin="+"/>
+<wire x1="152.4" y1="137.16" x2="134.62" y2="137.16" width="0.1524" layer="91"/>
+<junction x="152.4" y="137.16"/>
 </segment>
 </net>
@@
 </segment>
 </net>
+</nets>
+</sheet>
+<sheet>
+<plain>
+</plain>
+<instances>
+<instance part="FRAME3" gate="G$1" x="0" y="0"/>
+<instance part="FRAME3" gate="G$2" x="147.32" y="0"/>
+<instance part="U3" gate="G$1" x="48.26" y="68.58"/>
+<instance part="A1" gate="G$1" x="81.28" y="93.98"/>
+<instance part="A2" gate="G$1" x="96.52" y="93.98"/>
+<instance part="A3" gate="G$1" x="109.22" y="93.98"/>
+<instance part="J4" gate="G$1" x="142.24" y="142.24"/>
+<instance part="P+6" gate="VCC" x="124.46" y="152.4"/>
+<instance part="GND1" gate="1" x="124.46" y="132.08"/>
+</instances>
+<busses>
+</busses>
+<nets>
+<net name="GND" class="0">
+<segment>
+<pinref part="J4" gate="G$1" pin="GND"/>
+<pinref part="GND1" gate="1" pin="GND"/>
+<wire x1="129.54" y1="137.16" x2="124.46" y2="137.16" width="0.1524" layer="91"/>
+<wire x1="124.46" y1="137.16" x2="124.46" y2="134.62" width="0.1524" layer="91"/>
+</segment>
+</net>
+<net name="VCC" class="0">
+<segment>
+<pinref part="J4" gate="G$1" pin="VCC"/>
+<pinref part="P+6" gate="VCC" pin="VCC"/>
+<wire x1="129.54" y1="147.32" x2="124.46" y2="147.32" width="0.1524" layer="91"/>
+<wire x1="124.46" y1="147.32" x2="124.46" y2="149.86" width="0.1524" layer="91"/>
+</segment>
+</net>

Commit message: tag coming along
Parts:
- D1: value (none) -> GREEN
- D2: value (none) -> BLUE
Connections:
- new net N$1: A3.ANTENNA, U3.ANT1
- new net N$2: A2.ANTENNA, U3.ANT2
- new net N$3: A1.ANTENNA, U3.ANT3
- new net N$4: J4.SWDIO, U3.SWDIO
- new net N$7: J4.SWDCLK, U3.SWDCLK
- new net N$8: J4.!RESET, U3.!RESET
- net DW_INT: now also U3.INTERRUPT
- net GND: now also U3.GND
- net I2C_SCL: now also U3.SCL
- net I2C_SDA: now also U3.SDA
- net N$6: now also U5.P17; no longer U5.P24
- net VCC: now also U3.VCC
Other:
- moved on the sheet: A1, A2, A3, D1, D2, J4, R1, R12, R2, R3

Commit message: renamed parts, added bom
Parts:
- removed C15: 0.1uF, passives:CAPACITOR
- removed C17: 0.47uF, passives:CAPACITOR
- removed C18: 1uF, passives:CAPACITOR
- removed L3: 10uH, passives:INDUCTOR0603
- removed R10: 2k 1%, passives:RESISTOR0402_RES
- removed R12: 1k, passives:RESISTOR0402_RES
- removed R14: 2.2M, passives:RESISTOR0402_RES
- removed R15: 10M, passives:RESISTOR0402_RES
- removed U$3, U$4: BAT_HOLE, connector:BAT_HOLE
- removed U5: NRF51822QF, chips:NRF51822QF
- added C12: 1uF, passives:CAPACITOR
- added C5: 2.2nF, passives:CAPACITOR
- added C9: 0.1uF, passives:CAPACITOR
- added J1: TC2030-JLINK-NL, connector:TC2030-JLINK-NL
- added J5: BAT_HOLE, connector:BAT_HOLE
- added L2: 10uH, passives:INDUCTOR0603
- added R4, R5: 10k, passives:RESISTOR0402_RES
- added R7: 2.2M, passives:RESISTOR0402_RES
- added R8: 10M, passives:RESISTOR0402_RES
- added U1: NRF51822QF, chips:NRF51822QF
- C10: value 47nF -> 0.1uF
- C11: value 0.1uF -> 0.47uF
- C4: value 0.1uF -> 1nF
- C6: value 1nF -> 47nF
- C7: value 100nF -> 0.1uF
- C8: value 2.2nF -> 0.1uF
- J4: value TC2030-JLINK-NL -> BAT_HOLE; device connector:TC2030-JLINK-NL -> connector:BAT_HOLE
- R1, R2: value 10k -> 1k
- R3: value 1k -> 2k 1%
- U2: value LTC4065 -> TRIPOINT; device chips:LTC4065 -> tripoint:TRIPOINT
- U3: value TRIPOINT -> LTC4065; device tripoint:TRIPOINT -> chips:LTC4065
Connections:
- net !CHRG: now also R2.1; no longer R12.1
- net !CHRG1: now also R1.1; no longer R3.1
- net AVDD: now also C12.1, C4.1, U1.AVDD; no longer C13.1, C6.1, U5.AVDD
- net BATIN: now also C9.2, R7.2, R8.1, U1.P01/AIN2; no longer C15.2, R14.2, R15.1
- net DCC: now also L2.2, U1.DCC; no longer L3.2, U5.DCC
- net DW_INT: now also U1.P25, U2.INTERRUPT; no longer U3.INTERRUPT, U5.P25
- net GND: now also C12.2, C5.2, C9.1, J1.GND, J4.-, J5.-, R3.1, R7.1, U1.GND, U3.!EN; no longer C15.1, C17.2, C18.2, J4.GND, R10.1, R14.1, U$3.-, U$4.-, U2.!EN, U5.GND
- net I2C_SCL: now also R5.1, U1.P28, U2.SCL; no longer R2.1, U3.SCL, U5.P28
- net I2C_SDA: now also R4.1, U1.P29, U2.SDA; no longer R1.1, U3.SDA, U5.P29
- net N$1: now also U2.ANT1; no longer U3.ANT1
- net N$10: now also U1.XC2; no longer U5.XC2
- net N$13: now also R3.2, U3.PROG; no longer R10.2, U2.PROG
- net N$15: now also C6.1, U1.DEC2; no longer C10.1, U5.DEC2
- net N$17: now also U1.DEC1; no longer U5.DEC1
- net N$18: now also U1.ANT1; no longer U5.ANT1
- net N$19: now also U1.ANT2; no longer U5.ANT2
- net N$2: now also U2.ANT2; no longer U3.ANT2
- net N$20: now also C5.1, U1.VDD_PA; no longer C8.1, U5.VDD_PA
- net N$3: now also U2.ANT3; no longer U3.ANT3
- net N$37: now also L2.1; no longer L3.1
- net N$4: now also J2.SWDIO, U2.SWDIO; no longer J4.SWDIO, U3.SWDIO
- net N$5: now also U3.!CHRG; no longer U2.!CHRG
- net N$6: now also U1.P17; no longer U5.P17
- net N$7: now also J2.SWDCLK, U2.SWDCLK; no longer J4.SWDCLK, U3.SWDCLK
- net N$8: now also J2.!RESET, U2.!RESET; no longer J4.!RESET, U3.!RESET
- net N$9: now also U1.XC1; no longer U5.XC1
- net SWDCLK: now also J1.SWDCLK, U1.SWDCLK; no longer J2.SWDCLK, U5.SWDCLK
- net SWDIO/!RESET: now also J1.SWDIO, U1.SWDIO/!RESET; no longer J2.SWDIO, U5.SWDIO/!RESET
- net VBAT: now also C10.1, J4.+, J5.+, R8.2, U3.BAT; no longer C4.1, R15.2, U$3.+, U$4.+, U2.BAT
- net VCC: now also C8.1, J1.VCC, R4.2, R5.2, U1.VDD, U2.VCC; no longer C17.1, J4.VCC, R2.2, R3.2, U3.VCC, U5.VDD
- net VUSB: now also C13.1, R2.2, U3.VCC; no longer C18.1, R12.2, U2.VCC
Other:
- note added: "DecaWave"
- note added: "Power Supply and Charging"
- note added: "nRF51822 BLE"

Commit message: added debug pads
Parts:
- added TP1, TP2, TP3, TP4: TPTP06SQ, testpad:TPTP06SQ
Connections:
- net DW_INT: now also TP3.TP
- net GND: now also TP4.TP
- net I2C_SCL: now also TP1.TP
- net I2C_SDA: now also TP2.TP
Changed lines of the file:
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@@
 <attribute name="AUTHOR" value="Brad Campbell"/>
 <attribute name="REV" value="A"/>
-<attribute name="TITLE" value="Tritag"/>
+<attribute name="TITLE" value="PolyTag"/>
 </attributes>
 <variantdefs>
@@
 <part name="GND2" library="supply1" deviceset="GND" device=""/>
 <part name="SUPPLY8" library="supply1" deviceset="GND" device=""/>
+<part name="TP2" library="testpad" deviceset="TP" device="TP06SQ"/>
+<part name="TP1" library="testpad" deviceset="TP" device="TP06SQ"/>
+<part name="TP3" library="testpad" deviceset="TP" device="TP06SQ"/>
+<part name="TP4" library="testpad" deviceset="TP" device="TP06SQ"/>
 </parts>
 <sheets>
@@
 <instance part="GND2" gate="1" x="142.24" y="93.98"/>
 <instance part="LOGO1" gate="G$1" x="231.14" y="172.72"/>
+<instance part="TP2" gate="G$1" x="134.62" y="116.84" rot="R180"/>
+<instance part="TP1" gate="G$1" x="129.54" y="116.84" rot="R180"/>
+<instance part="TP3" gate="G$1" x="139.7" y="116.84" rot="R180"/>
+<instance part="TP4" gate="G$1" x="137.16" y="106.68"/>
 </instances>
 <busses>
@@
 <pinref part="U2" gate="G$1" pin="GND"/>
 <wire x1="144.78" y1="104.14" x2="142.24" y2="104.14" width="0.1524" layer="91"/>
-<wire x1="142.24" y1="104.14" x2="142.24" y2="96.52" width="0.1524" layer="91"/>
+<wire x1="142.24" y1="104.14" x2="142.24" y2="101.6" width="0.1524" layer="91"/>
 <pinref part="GND2" gate="1" pin="GND"/>
+<pinref part="TP4" gate="G$1" pin="TP"/>
+<wire x1="142.24" y1="101.6" x2="142.24" y2="96.52" width="0.1524" layer="91"/>
+<wire x1="137.16" y1="104.14" x2="137.16" y2="101.6" width="0.1524" layer="91"/>
+<wire x1="137.16" y1="101.6" x2="142.24" y2="101.6" width="0.1524" layer="91"/>
+<junction x="142.24" y="101.6"/>
 </segment>
 </net>
@@
 <segment>
 <pinref part="U2" gate="G$1" pin="INTERRUPT"/>
-<wire x1="144.78" y1="124.46" x2="111.76" y2="124.46" width="0.1524" layer="91"/>
+<wire x1="144.78" y1="124.46" x2="139.7" y2="124.46" width="0.1524" layer="91"/>
+<wire x1="139.7" y1="124.46" x2="111.76" y2="124.46" width="0.1524" layer="91"/>
 <wire x1="111.76" y1="124.46" x2="111.76" y2="93.98" width="0.1524" layer="91"/>
 <label x="93.98" y="81.28" size="1.27" layer="95" xref="yes"/>
@@
 <wire x1="91.44" y1="93.98" x2="91.44" y2="81.28" width="0.1524" layer="91"/>
 <junction x="91.44" y="81.28"/>
+<pinref part="TP3" gate="G$1" pin="TP"/>
+<wire x1="139.7" y1="119.38" x2="139.7" y2="124.46" width="0.1524" layer="91"/>
+<junction x="139.7" y="124.46"/>
 </segment>
 </net>
@@
 <pinref part="U2" gate="G$1" pin="SDA"/>
 <wire x1="109.22" y1="129.54" x2="119.38" y2="129.54" width="0.1524" layer="91"/>
-<wire x1="119.38" y1="129.54" x2="144.78" y2="129.54" width="0.1524" layer="91"/>
+<wire x1="119.38" y1="129.54" x2="134.62" y2="129.54" width="0.1524" layer="91"/>
+<wire x1="134.62" y1="129.54" x2="144.78" y2="129.54" width="0.1524" layer="91"/>
 <wire x1="119.38" y1="137.16" x2="119.38" y2="129.54" width="0.1524" layer="91"/>
 <junction x="119.38" y="137.16"/>
 <junction x="119.38" y="129.54"/>
+<pinref part="TP2" gate="G$1" pin="TP"/>
+<wire x1="134.62" y1="119.38" x2="134.62" y2="129.54" width="0.1524" layer="91"/>
+<junction x="134.62" y="129.54"/>
 </segment>
 </net>
@@
 <label x="129.54" y="137.16" size="1.27" layer="95" xref="yes"/>
 <pinref part="U2" gate="G$1" pin="SCL"/>
-<wire x1="144.78" y1="132.08" x2="127" y2="132.08" width="0.1524" layer="91"/>
+<wire x1="144.78" y1="132.08" x2="129.54" y2="132.08" width="0.1524" layer="91"/>
+<wire x1="129.54" y1="132.08" x2="127" y2="132.08" width="0.1524" layer="91"/>
 <wire x1="127" y1="132.08" x2="106.68" y2="132.08" width="0.1524" layer="91"/>
 <wire x1="106.68" y1="132.08" x2="106.68" y2="73.66" width="0.1524" layer="91"/>
@@
 <junction x="127" y="137.16"/>
 <junction x="127" y="132.08"/>
-</segment>
-</net>
+<pinref part="TP1" gate="G$1" pin="TP"/>
+<wire x1="129.54" y1="119.38" x2="129.54" y2="132.08" width="0.1524" layer="91"/>
+<junction x="129.54" y="132.08"/>
+</segment>
+</net>
