File: pcb/anchor/rev_a/anchor.brd (EAGLE design)
At the start: 53.3 x 63.2 mm, 3 parts, among them J1 CUI_PJ-069B-SMT-TR, U1 TRIPOINT

Commit message: much farther on anchor
Parts:
- added A1, A2, A3: TAIYO-YUDEN-AH086M, chips:TAIYO-YUDEN-AH086M
- added C1, C2: 47pF, passives:0402_CAP
- added C3, C5: 10uF, passives:0603_CAP
- added C4: 10pF, passives:0402_CAP
- added J2: CUI_PJ-069B-SMT-TR, connector:PJ-069B-SMT-TR
- added L1: 1uH, SparkFun-Passives:1210
- added R1, R2: 27, passives:0402_RES
- added R3: 680k, passives:0402_RES
- added R4: 120k, passives:0402_RES
- added R5, R6: 100, passives:0402_RES
- added U2: TPS62065, chips:S-PWSON-N8
- added U4: FTDI234XD, chips:DFN-12/3MM
- J1: value CUI_PJ-069B-SMT-TR -> USB_C_JAE_DX07S024JJ2; device connector:PJ-069B-SMT-TR -> connector:DX07S024JJ2
- moved J1 57.0 mm to (-12.1, 22.9), flipped to the bottom, turned to 180 degrees
- moved E_1 46.3 mm to (11.2, -23.3), turned to 30 degrees
- moved U1 37.9 mm to (0.00, 0.00)
Connections:
- new net D+: C2.1, J1.A6, J1.B6, R2.1
- new net D-: C1.1, J1.A7, J1.B7, R1.1
- new net EDISON_UART_RX: E_1.22, R5.2
- new net EDISON_UART_TX: E_1.27, R6.2
- new net GND: C1.2, C2.2, C3.2, C5.2, E_1.1, E_1.11, E_1.13, E_1.15, E_1.5, E_1.9, J1.A1, J1.A12, J1.B1, J1.B12, R4.1, U2.1, U2.3, U2.6, U2.P$1, U4.13, U4.5
- new net N$1: L1.1, U2.2
- new net N$2: R5.1, U4.7
- new net N$6: R1.2, U4.1
- new net N$7: R2.2, U4.12
- new net N$8: C4.2, R3.1, R4.2, U2.4
- new net N$9: R6.1, U4.10
- new net VBUS: C5.1, J1.A4, J1.A9, J1.B4, J1.B9, U2.5, U2.7, U2.8, U4.4
- new net VCC: C3.1, C4.1, E_1.2, E_1.4, E_1.6, L1.2, R3.2
Routing:
- net N$3: track 0.00 -> 23.7 mm
- net N$4: track 0.00 -> 23.6 mm
- net N$5: track 0.00 -> 23.5 mm
- net VBUS: track 0.00 -> 8.64 mm
- net D+: track 0.00 -> 7.66 mm
- net D-: track 0.00 -> 5.88 mm, vias 0 -> 2
- net GND: track 0.00 -> 3.51 mm
- net N$6: track 0.00 -> 1.41 mm
- net N$7: track 0.00 -> 1.25 mm
Other:
- board size 53.3 x 63.2 mm -> 68 x 61 mm

Commit message: added some to anchor
Parts:
- added LOGO1: UMICH_SOLID_MEDIUM, logos:UMICH_SOLID_200MIL
- added R7, R8: 10k, passives:0402_RES
- moved R4 3.81 mm to (6.55, 21.2)
- moved C3 3.81 mm to (5.00, 17.9)
- moved L1 3.81 mm to (3.05, 21.1)
- moved U2 3.81 mm to (2.54, 17.8)
- moved C4 3.81 mm to (8.79, 21.2)
- moved C5 3.81 mm to (0.38, 17.8)
- moved R3 3.81 mm to (7.59, 21.2)
- moved R2 2.54 mm to (-8.00, 9.91)
- moved U4 2.54 mm to (-5.21, 11.3)
- moved C1 2.54 mm to (-8.10, 13.4)
- moved C2 2.54 mm to (-10.7, 13.9)
- moved J1 2.54 mm to (-9.53, 22.9)
- moved R1 2.54 mm to (-8.13, 12.7)
- moved R5 1.80 mm to (6.35, -5.08), turned to 180 degrees
- moved R6 1.27 mm to (6.35, -6.35), turned to 180 degrees
Connections:
- new net SCL: E_1.41, R8.2
- new net SDA: E_1.43, R7.2
- net VCC: now also R7.1, R8.1
Routing:
- net N$9: track 0.00 -> 21.4 mm
- net N$2: track 0.00 -> 19.6 mm
- net EDISON_UART_TX: track 0.00 -> 14.1 mm, vias 0 -> 2
- net EDISON_UART_RX: track 0.00 -> 9.08 mm
- added copper zone on layer 1, net GND
Other:
- outline, holes or cut-outs redrawn

Commit message: routed anchor
Parts:
- J2: value CUI_PJ-069B-SMT-TR -> TC2030-JLINK-NL; device connector:PJ-069B-SMT-TR -> connector:TC2030-IDC-NL
- moved J2 94.4 mm to (-20.3, -5.69), turned to 300 degrees
- moved R5 6.63 mm to (12.0, -8.56), turned to 240 degrees
- moved R6 5.47 mm to (11.0, -9.19), turned to 240 degrees
- moved C5 1.71 mm to (-1.32, 17.9)
- moved C3 1.71 mm to (3.30, 18.0)
- moved L1 1.71 mm to (1.35, 21.2)
- moved U2 1.71 mm to (0.84, 17.9)
- moved R4 1.55 mm to (5.00, 21.1), turned to 90 degrees
- moved R3 1.45 mm to (6.15, 21.1)
- moved C4 1.40 mm to (7.39, 21.1)
- moved R2 1.38 mm to (-8.10, 11.3)
- moved C2 0.66 mm to (-10.7, 13.3)
- moved R1 0.36 mm to (-8.10, 12.3)
Connections:
- new net DW_INT: E_1.48, U1.38
- new net N$10: A2.A, U1.9
- new net N$11: A1.A, U1.26
- new net N$12: A3.A, U1.43
- new net N$13: J2.4, U1.29
- new net N$14: J2.3, U1.30
- new net N$5: J2.2, U1.28
- net GND: now also J2.5, U1.10, U1.18, U1.25, U1.27, U1.42, U1.44, U1.8
- net SCL: now also U1.37
- net SDA: now also U1.36
- net VCC: now also J2.1, U1.17
Routing:
- net VCC: track 0.00 -> 92.5 mm, vias 0 -> 8
- net GND: track 3.51 -> 67.3 mm, vias 0 -> 20
- net SDA: track 0.00 -> 39.5 mm, vias 0 -> 3
- net SCL: track 0.00 -> 36.7 mm, vias 0 -> 3
- net DW_INT: track 0.00 -> 27.9 mm, vias 0 -> 1
- net N$3: track 23.7 -> 0.00 mm
- net N$4: track 23.6 -> 0.00 mm
- net N$11: track 0.00 -> 17.4 mm
- net N$10: track 0.00 -> 17.4 mm
- net N$12: track 0.00 -> 17.4 mm
- net N$14: track 0.00 -> 13.7 mm, vias 0 -> 2
- net N$13: track 0.00 -> 12.0 mm
- net VBUS: track 8.64 -> 19.8 mm, vias 0 -> 2
- net N$5: track 23.5 -> 13.6 mm
- net N$8: track 0.00 -> 8.52 mm, vias 0 -> 2
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- added copper zone on layer 16, net GND
- added copper zone on layer 16, net N$1
- added copper zone on layer 16, net VBUS
- added copper zone on layer 16, net VCC
