File: pcb/anchor/rev_a/anchor.sch (EAGLE design)
At the start: 3 parts, among them J1 CUI_PJ-069B-SMT-TR, U1 TRIPOINT

Commit message: much farther on anchor
Parts:
- added A1, A2, A3: TAIYO-YUDEN-AH086M, chips:TAIYO-YUDEN-AH086M
- added C1, C2: 47pF, passives:CAPACITOR
- added C3, C5: 10uF, passives:CAPACITOR0603_CAP
- added C4: 10pF, passives:CAPACITOR
- added J2: CUI_PJ-069B-SMT-TR, connector:CUI_PJ-069B-SMT-TR
- added L1: 1uH, SparkFun-Passives:INDUCTOR1210
- added R1, R2: 27, passives:RESISTOR0402_RES
- added R3: 680k, passives:RESISTOR0402_RES
- added R4: 120k, passives:RESISTOR0402_RES
- added R5, R6: 100, passives:RESISTOR0402_RES
- added U2: TPS62065, chips:TPS62065
- added U4: FTDI234XD, chips:FTDI234XD
- J1: value CUI_PJ-069B-SMT-TR -> USB_C_JAE_DX07S024JJ2; device connector:CUI_PJ-069B-SMT-TR -> connector:USB_C_JAE_DX07S024JJ2
Connections:
- new net D+: C2.1, J1.D+, R2.1
- new net D-: C1.1, J1.D-, R1.1
- new net EDISON_UART_RX: E_1_UART_2.GP134_UART_2_RX, R5.2
- new net EDISON_UART_TX: E_1_UART_2.GP135_UART_2_TX, R6.2
- new net GND: C1.2, C2.2, C3.2, C5.2, E_1_BASIC.GND@1, E_1_BASIC.GND@2, E_1_BASIC.GND@3, E_1_BASIC.GND@4, E_1_BASIC.GND@5, E_1_BASIC.GND@6, J1.GND, R4.1, U2.AGND, U2.PG, U2.PGND, U4.GND
- new net N$1: L1.1, U2.SW
- new net N$2: R5.1, U4.TXD
- new net N$6: R1.2, U4.USBDM
- new net N$7: R2.2, U4.USBDP
- new net N$8: C4.2, R3.1, R4.2, U2.FB
- new net N$9: R6.1, U4.RXD
- new net VBUS: C5.1, J1.VBUS, U2.AVIN, U2.EN, U2.PVIN, U4.VCC
- new net VCC: C3.1, C4.1, E_1_BASIC.VSYS@1, E_1_BASIC.VSYS@2, E_1_BASIC.VSYS@3, L1.2, R3.2

Commit message: added some to anchor
Parts:
- added LOGO1: UMICH_SOLID_MEDIUM, logos:UMICH_SOLID_MEDIUM
- added R7, R8: 10k, passives:RESISTOR0402_RES
Connections:
- new net SCL: E_1_I2C_1.GP19_I2C_1_SCL, R8.2
- new net SDA: E_1_I2C_1.GP20_I2C_1_SDA, R7.2
- net VCC: now also R7.1, R8.1
Other:
- moved on the sheet: E_1_I2C_1, E_1_I2C_6
Changed lines of the file:
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@@
 <schematic xreflabel="%F%N/%S.%C%R" xrefpart="/%S.%C%R">
 <attributes>
+<attribute name="AUTHOR" value="Brad Campbell"/>
+<attribute name="REV" value="A"/>
 </attributes>
 <variantdefs>
@@
 <part name="P+2" library="supply1" deviceset="VCC" device=""/>
 <part name="GND9" library="supply1" deviceset="GND" device=""/>
+<part name="R7" library="passives" deviceset="RESISTOR" device="0402_RES" value="10k"/>
+<part name="R8" library="passives" deviceset="RESISTOR" device="0402_RES" value="10k"/>
+<part name="P+3" library="supply1" deviceset="VCC" device=""/>
+<part name="P+4" library="supply1" deviceset="VCC" device=""/>
+<part name="LOGO1" library="logos" deviceset="UMICH_SOLID" device="_MEDIUM"/>
 </parts>
 <sheets>
@@
 <instance part="E_1" gate="_BASIC" x="30.48" y="165.1"/>
 <instance part="E_1" gate="_GPIO" x="30.48" y="111.76"/>
-<instance part="E_1" gate="_I2C_1" x="91.44" y="165.1"/>
-<instance part="E_1" gate="_I2C_6" x="91.44" y="137.16"/>
+<instance part="E_1" gate="_I2C_1" x="91.44" y="132.08"/>
+<instance part="E_1" gate="_I2C_6" x="91.44" y="116.84"/>
 <instance part="E_1" gate="_I2S" x="91.44" y="101.6"/>
 <instance part="E_1" gate="_SD" x="91.44" y="68.58"/>
@@
 <instance part="P+2" gate="VCC" x="25.4" y="172.72"/>
 <instance part="GND9" gate="1" x="25.4" y="124.46"/>
+<instance part="R7" gate="G$1" x="83.82" y="139.7" smashed="yes" rot="R270">
+<attribute name="NAME" x="85.3186" y="143.51" size="1.778" layer="95" rot="R270"/>
+<attribute name="VALUE" x="85.598" y="138.43" size="1.778" layer="96" rot="R270"/>
+</instance>
+<instance part="R8" gate="G$1" x="78.74" y="139.7" smashed="yes" rot="R270">
+<attribute name="NAME" x="75.1586" y="143.51" size="1.778" layer="95" rot="R270"/>
+<attribute name="VALUE" x="75.438" y="138.43" size="1.778" layer="96" rot="R270"/>
+</instance>
+<instance part="P+3" gate="VCC" x="78.74" y="149.86"/>
+<instance part="P+4" gate="VCC" x="83.82" y="149.86"/>
+<instance part="LOGO1" gate="G$1" x="231.14" y="172.72"/>
 </instances>
 <busses>
@@
 <junction x="25.4" y="162.56"/>
 </segment>
+<segment>
+<pinref part="R8" gate="G$1" pin="1"/>
+<wire x1="78.74" y1="144.78" x2="78.74" y2="147.32" width="0.1524" layer="91"/>
+<pinref part="P+3" gate="VCC" pin="VCC"/>
+</segment>
+<segment>
+<pinref part="R7" gate="G$1" pin="1"/>
+<wire x1="83.82" y1="144.78" x2="83.82" y2="147.32" width="0.1524" layer="91"/>
+<pinref part="P+4" gate="VCC" pin="VCC"/>
+</segment>
 </net>
 <net name="GND" class="0">
@@
 </segment>
 </net>
+<net name="SCL" class="0">
+<segment>
+<pinref part="R8" gate="G$1" pin="2"/>
+<wire x1="78.74" y1="134.62" x2="78.74" y2="129.54" width="0.1524" layer="91"/>
+<pinref part="E_1" gate="_I2C_1" pin="GP19_I2C_1_SCL"/>
+<wire x1="78.74" y1="129.54" x2="88.9" y2="129.54" width="0.1524" layer="91"/>
+<wire x1="78.74" y1="129.54" x2="73.66" y2="129.54" width="0.1524" layer="91"/>
+<junction x="78.74" y="129.54"/>
+<label x="73.66" y="129.54" size="1.27" layer="95" rot="R180" xref="yes"/>
+</segment>
+</net>
+<net name="SDA" class="0">
+<segment>
+<pinref part="R7" gate="G$1" pin="2"/>
+<wire x1="83.82" y1="134.62" x2="83.82" y2="132.08" width="0.1524" layer="91"/>
+<pinref part="E_1" gate="_I2C_1" pin="GP20_I2C_1_SDA"/>
+<wire x1="83.82" y1="132.08" x2="88.9" y2="132.08" width="0.1524" layer="91"/>
+<wire x1="83.82" y1="132.08" x2="73.66" y2="132.08" width="0.1524" layer="91"/>
+<junction x="83.82" y="132.08"/>
+<label x="73.66" y="132.08" size="1.27" layer="95" rot="R180" xref="yes"/>
+</segment>
+</net>

Commit message: some misc changes to anchor
Parts:
- L1: DIGIKEY (none) -> 490-10767-1-ND
Changed lines of the file:
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@@
 <part name="U2" library="chips" deviceset="TPS62065" device=""/>
 <part name="GND5" library="supply1" deviceset="GND" device=""/>
-<part name="L1" library="SparkFun-Passives" deviceset="INDUCTOR" device="1210" value="1uH"/>
+<part name="L1" library="SparkFun-Passives" deviceset="INDUCTOR" device="1210" value="1uH">
+<attribute name="DIGIKEY" value="490-10767-1-ND"/>
+</part>
 <part name="R3" library="passives" deviceset="RESISTOR" device="0402_RES" value="680k"/>
 <part name="R4" library="passives" deviceset="RESISTOR" device="0402_RES" value="120k"/>
@@
 <instance part="U2" gate="G$1" x="66.04" y="55.88"/>
 <instance part="GND5" gate="1" x="50.8" y="30.48"/>
-<instance part="L1" gate="G$1" x="88.9" y="63.5" rot="R90"/>
+<instance part="L1" gate="G$1" x="88.9" y="63.5" rot="R90">
+<attribute name="DIGIKEY" x="88.9" y="63.5" size="3.81" layer="96" rot="R90" align="bottom-center" display="off"/>
+</instance>
 <instance part="R3" gate="G$1" x="99.06" y="55.88" smashed="yes" rot="R90">
 <attribute name="NAME" x="102.6414" y="52.07" size="1.778" layer="95" rot="R90"/>

Commit message: routed anchor
Parts:
- J2: value CUI_PJ-069B-SMT-TR -> TC2030-JLINK-NL; device connector:CUI_PJ-069B-SMT-TR -> connector:TC2030-JLINK-NL
Connections:
- new net DW_INT: E_1_GPIO.GP14, U1.INTERRUPT
- new net N$10: A2.ANTENNA, U1.ANT1
- new net N$11: A1.ANTENNA, U1.ANT2
- new net N$12: A3.ANTENNA, U1.ANT3
- new net N$13: J2.SWDCLK, U1.SWDCLK
- new net N$14: J2.!RESET, U1.!RESET
- new net N$5: J2.SWDIO, U1.SWDIO
- net GND: now also J2.GND, U1.GND
- net SCL: now also U1.SCL
- net SDA: now also U1.SDA
- net VCC: now also J2.VCC, U1.VCC
Other:
- moved on the sheet: E_1_I2C_6, E_1_I2S, E_1_SD, E_1_SPI, E_1_UART_1, E_1_UART_2, E_1_USB
Changed lines of the file:
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@@
 <attribute name="AUTHOR" value="Brad Campbell"/>
 <attribute name="REV" value="A"/>
+<attribute name="TITLE" value="PolyAnchor"/>
 </attributes>
 <variantdefs>
@@
 <part name="A2" library="chips" deviceset="TAIYO-YUDEN-AH086M" device=""/>
 <part name="A3" library="chips" deviceset="TAIYO-YUDEN-AH086M" device=""/>
-<part name="J2" library="connector" deviceset="CUI_PJ-069B-SMT-TR" device=""/>
 <part name="J1" library="connector" deviceset="USB_C_JAE_DX07S024JJ2" device=""/>
 <part name="FRAME3" library="frames" deviceset="LETTER_L" device=""/>
@@
 <part name="P+4" library="supply1" deviceset="VCC" device=""/>
 <part name="LOGO1" library="logos" deviceset="UMICH_SOLID" device="_MEDIUM"/>
+<part name="P+5" library="supply1" deviceset="VCC" device=""/>
+<part name="GND10" library="supply1" deviceset="GND" device=""/>
+<part name="J2" library="connector" deviceset="TC2030-JLINK" device="-NL"/>
+<part name="P+6" library="supply1" deviceset="VCC" device=""/>
+<part name="GND11" library="supply1" deviceset="GND" device=""/>
 </parts>
 <sheets>
@@
 <instance part="E_1" gate="_GPIO" x="30.48" y="111.76"/>
 <instance part="E_1" gate="_I2C_1" x="91.44" y="132.08"/>
-<instance part="E_1" gate="_I2C_6" x="91.44" y="116.84"/>
-<instance part="E_1" gate="_I2S" x="91.44" y="101.6"/>
-<instance part="E_1" gate="_SD" x="91.44" y="68.58"/>
-<instance part="E_1" gate="_SPI" x="139.7" y="165.1"/>
-<instance part="E_1" gate="_UART_1" x="139.7" y="132.08"/>
-<instance part="E_1" gate="_UART_2" x="177.8" y="104.14"/>
-<instance part="E_1" gate="_USB" x="144.78" y="81.28"/>
+<instance part="E_1" gate="_I2C_6" x="63.5" y="7.62"/>
+<instance part="E_1" gate="_I2S" x="40.64" y="38.1"/>
+<instance part="E_1" gate="_SD" x="10.16" y="35.56"/>
+<instance part="E_1" gate="_SPI" x="96.52" y="15.24"/>
+<instance part="E_1" gate="_UART_1" x="66.04" y="27.94"/>
+<instance part="E_1" gate="_UART_2" x="88.9" y="101.6"/>
+<instance part="E_1" gate="_USB" x="40.64" y="17.78"/>
 <instance part="P+2" gate="VCC" x="25.4" y="172.72"/>
 <instance part="GND9" gate="1" x="25.4" y="124.46"/>
@@
 <instance part="P+4" gate="VCC" x="83.82" y="149.86"/>
 <instance part="LOGO1" gate="G$1" x="231.14" y="172.72"/>
+<instance part="U1" gate="G$1" x="165.1" y="124.46"/>
+<instance part="A1" gate="G$1" x="208.28" y="147.32"/>
+<instance part="A2" gate="G$1" x="198.12" y="149.86"/>
+<instance part="A3" gate="G$1" x="218.44" y="144.78"/>
+<instance part="P+5" gate="VCC" x="137.16" y="152.4"/>
+<instance part="GND10" gate="1" x="139.7" y="96.52"/>
+<instance part="J2" gate="G$1" x="208.28" y="109.22" rot="MR0"/>
+<instance part="P+6" gate="VCC" x="223.52" y="121.92"/>
+<instance part="GND11" gate="1" x="223.52" y="96.52"/>
 </instances>
 <busses>
@@
 <segment>
 <pinref part="E_1" gate="_UART_2" pin="GP135_UART_2_TX"/>
-<wire x1="175.26" y1="104.14" x2="172.72" y2="104.14" width="0.1524" layer="91"/>
-<label x="172.72" y="104.14" size="1.27" layer="95" rot="R180" xref="yes"/>
+<wire x1="86.36" y1="101.6" x2="83.82" y2="101.6" width="0.1524" layer="91"/>
+<label x="83.82" y="101.6" size="1.27" layer="95" rot="R180" xref="yes"/>
 </segment>
 </net>
@@
 <segment>
 <pinref part="E_1" gate="_UART_2" pin="GP134_UART_2_RX"/>
-<wire x1="175.26" y1="101.6" x2="172.72" y2="101.6" width="0.1524" layer="91"/>
-<label x="172.72" y="101.6" size="1.27" layer="95" rot="R180" xref="yes"/>
+<wire x1="86.36" y1="99.06" x2="83.82" y2="99.06" width="0.1524" layer="91"/>
+<label x="83.82" y="99.06" size="1.27" layer="95" rot="R180" xref="yes"/>
 </segment>
 </net>
@@
 <wire x1="83.82" y1="144.78" x2="83.82" y2="147.32" width="0.1524" layer="91"/>
 <pinref part="P+4" gate="VCC" pin="VCC"/>
+</segment>
+<segment>
+<pinref part="P+5" gate="VCC" pin="VCC"/>
+<wire x1="137.16" y1="149.86" x2="137.16" y2="139.7" width="0.1524" layer="91"/>
+<pinref part="U1" gate="G$1" pin="VCC"/>
+<wire x1="137.16" y1="139.7" x2="142.24" y2="139.7" width="0.1524" layer="91"/>
+</segment>
+<segment>
+<pinref part="J2" gate="G$1" pin="VCC"/>
+<wire x1="220.98" y1="114.3" x2="223.52" y2="114.3" width="0.1524" layer="91"/>
+<wire x1="223.52" y1="114.3" x2="223.52" y2="119.38" width="0.1524" layer="91"/>
+<pinref part="P+6" gate="VCC" pin="VCC"/>
 </segment>
 </net>
@@
 <junction x="25.4" y="129.54"/>
 </segment>
+<segment>
+<pinref part="U1" gate="G$1" pin="GND"/>
+<wire x1="142.24" y1="106.68" x2="139.7" y2="106.68" width="0.1524" layer="91"/>
+<wire x1="139.7" y1="106.68" x2="139.7" y2="99.06" width="0.1524" layer="91"/>
+<pinref part="GND10" gate="1" pin="GND"/>
+</segment>
+<segment>
+<pinref part="J2" gate="G$1" pin="GND"/>
+<wire x1="220.98" y1="104.14" x2="223.52" y2="104.14" width="0.1524" layer="91"/>
+<wire x1="223.52" y1="104.14" x2="223.52" y2="99.06" width="0.1524" layer="91"/>
+<pinref part="GND11" gate="1" pin="GND"/>
+</segment>
 </net>
 <net name="SCL" class="0">
@@
 <label x="73.66" y="129.54" size="1.27" layer="95" rot="R180" xref="yes"/>
 </segment>
+<segment>
+<pinref part="U1" gate="G$1" pin="SCL"/>
+<wire x1="142.24" y1="134.62" x2="139.7" y2="134.62" width="0.1524" layer="91"/>
+<label x="139.7" y="134.62" size="1.27" layer="95" rot="R180" xref="yes"/>
+</segment>
 </net>
 <net name="SDA" class="0">
@@
 <junction x="83.82" y="132.08"/>
 <label x="73.66" y="132.08" size="1.27" layer="95" rot="R180" xref="yes"/>
+</segment>
+<segment>
+<pinref part="U1" gate="G$1" pin="SDA"/>
+<wire x1="142.24" y1="132.08" x2="139.7" y2="132.08" width="0.1524" layer="91"/>
+<label x="139.7" y="132.08" size="1.27" layer="95" rot="R180" xref="yes"/>
+</segment>
+</net>
+<net name="DW_INT" class="0">
+<segment>
+<label x="25.4" y="91.44" size="1.27" layer="95" rot="R180" xref="yes"/>
+<pinref part="E_1" gate="_GPIO" pin="GP14"/>
+<wire x1="27.94" y1="91.44" x2="25.4" y2="91.44" width="0.1524" layer="91"/>
+</segment>
+<segment>
+<pinref part="U1" gate="G$1" pin="INTERRUPT"/>
+<wire x1="142.24" y1="127" x2="139.7" y2="127" width="0.1524" layer="91"/>
+<label x="139.7" y="127" size="1.27" layer="95" rot="R180" xref="yes"/>
+</segment>
+</net>
+<net name="N$10" class="0">
+<segment>
+<pinref part="U1" gate="G$1" pin="ANT1"/>
+<pinref part="A2" gate="G$1" pin="ANTENNA"/>
+<wire x1="185.42" y1="137.16" x2="198.12" y2="137.16" width="0.1524" layer="91"/>
+<wire x1="198.12" y1="137.16" x2="198.12" y2="144.78" width="0.1524" layer="91"/>
+</segment>
+</net>
+<net name="N$11" class="0">
+<segment>
+<pinref part="A1" gate="G$1" pin="ANTENNA"/>
+<wire x1="208.28" y1="142.24" x2="208.28" y2="132.08" width="0.1524" layer="91"/>
+<pinref part="U1" gate="G$1" pin="ANT2"/>
+<wire x1="208.28" y1="132.08" x2="185.42" y2="132.08" width="0.1524" layer="91"/>
+</segment>
+</net>
+<net name="N$12" class="0">
+<segment>
+<pinref part="U1" gate="G$1" pin="ANT3"/>
+<pinref part="A3" gate="G$1" pin="ANTENNA"/>
+<wire x1="185.42" y1="127" x2="218.44" y2="127" width="0.1524" layer="91"/>
+<wire x1="218.44" y1="127" x2="218.44" y2="139.7" width="0.1524" layer="91"/>
+</segment>
+</net>
+<net name="N$5" class="0">
+<segment>
+<pinref part="U1" gate="G$1" pin="SWDIO"/>
+<pinref part="J2" gate="G$1" pin="SWDIO"/>
+<wire x1="185.42" y1="114.3" x2="195.58" y2="114.3" width="0.1524" layer="91"/>
+</segment>
+</net>
+<net name="N$13" class="0">
+<segment>
+<pinref part="J2" gate="G$1" pin="SWDCLK"/>
+<pinref part="U1" gate="G$1" pin="SWDCLK"/>
+<wire x1="195.58" y1="111.76" x2="185.42" y2="111.76" width="0.1524" layer="91"/>
+</segment>
+</net>
+<net name="N$14" class="0">
+<segment>
+<pinref part="U1" gate="G$1" pin="!RESET"/>
+<wire x1="185.42" y1="109.22" x2="193.04" y2="109.22" width="0.1524" layer="91"/>
+<wire x1="193.04" y1="109.22" x2="193.04" y2="104.14" width="0.1524" layer="91"/>
+<pinref part="J2" gate="G$1" pin="!RESET"/>
+<wire x1="193.04" y1="104.14" x2="195.58" y2="104.14" width="0.1524" layer="91"/>
 </segment>
 </net>
@@
 <instance part="FRAME2" gate="G$1" x="0" y="0"/>
 <instance part="FRAME2" gate="G$2" x="147.32" y="0"/>
-<instance part="U1" gate="G$1" x="83.82" y="86.36"/>
-<instance part="A1" gate="G$1" x="116.84" y="119.38"/>
-<instance part="A2" gate="G$1" x="129.54" y="119.38"/>
-<instance part="A3" gate="G$1" x="142.24" y="119.38"/>
 </instances>
 <busses>
@@
 <instance part="GND8" gate="1" x="119.38" y="30.48"/>
 <instance part="P+1" gate="VCC" x="127" y="68.58"/>
-<instance part="J2" gate="G$1" x="180.34" y="137.16"/>
 <instance part="R5" gate="G$1" x="124.46" y="160.02" smashed="yes">
 <attribute name="NAME" x="120.65" y="161.5186" size="1.778" layer="95"/>
@@
 </sheet>
 </sheets>
+<errors>
+</errors>
 </schematic>
 </drawing>

Commit message: start working on ble notify
Changed lines of the file:
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@@
 <part name="FRAME1" library="frames" deviceset="LETTER_L" device=""/>
 <part name="E_1" library="Edison" deviceset="EDISON_CONNECTOR_SEGMENTED" device=""/>
-<part name="FRAME2" library="frames" deviceset="LETTER_L" device=""/>
 <part name="U1" library="tripoint" deviceset="TRIPOINT" device=""/>
 <part name="A1" library="chips" deviceset="TAIYO-YUDEN-AH086M" device=""/>
@@
 </nets>
 </sheet>
-<sheet>
-<plain>
-</plain>
-<instances>
-<instance part="FRAME2" gate="G$1" x="0" y="0"/>
-<instance part="FRAME2" gate="G$2" x="147.32" y="0"/>
-</instances>
-<busses>
-</busses>
-<nets>
-</nets>
-</sheet>
