File: pcb/protopoint-v1p1/protopoint.kicad_pcb (KiCad board)
At the start: 4 copper layers, 31.8 x 27.5 mm, 52 parts, among them T1 HHM1595A1, U1 STM32F031G6U6, U2 LXDC2HL, U3 DW1000, U4 SKY13317, U5 ProtoPoint_Module, X1 38.4M, X2 16M

Commit message: rename to tripoint...woah
Other:
- board text added: "TriPoint"
- board text removed: "ProtoPoint"
Changed lines of the file:
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@@
     (effects (font (size 1 1) (thickness 0.2)))
   )
-  (gr_text ProtoPoint (at 44.45 27.051) (layer F.SilkS)
+  (gr_text TriPoint (at 44.45 27.051) (layer F.SilkS)
     (effects (font (size 1 1) (thickness 0.2)))
   )
