File: pcb/protopoint-v1p1/protopoint.sch (KiCad schematic (older format))
At the start: 51 parts, among them T1 HHM1595A1, U1 STM32F031G6U6, U2 LXDC2HL, U3 DW1000, U4 SKY13317, U5 ProtoPoint_Module, X1 38.4M, X2 16M

Commit message: routing more signals out to castellations
Connections:
- net DW_IRQ: now also U5.39
- net SPI1_CLK: now also U5.22
- net SPI1_MISO: now also U5.21
- net SPI1_MOSI: now also U5.20
- net ~DW_RST: now also U5.24
- net ~SPI1_SS: now also U5.23
Changed lines of the file:
@@
 Text Label 3450 2650 0    60   ~ 0
 GPIO4
+Text Label 3150 5700 1    60   ~ 0
+DW_IRQ
+Text Label 3950 7150 0    60   ~ 0
+~SPI1_SS
+Text Label 3950 7250 0    60   ~ 0
+SPI1_CLK
+Text Label 3950 7350 0    60   ~ 0
+SPI1_MISO
+Text Label 3950 7450 0    60   ~ 0
+SPI1_MOSI
+Text Label 3950 7050 0    60   ~ 0
+~DW_RST
 $EndSCHEMATC

Commit message: adding support for external clock and sync
Connections:
- net DW_SYNC: now reaches U3.29 (SYNC)
- net DW_SYNC: now also U5.19
- net DW_XTAL1: now reaches C36.1, U3.3 (XTAL1), X2.3
- net DW_XTAL1: now also U5.49
Changed lines of the file:
@@
 Text Label 3950 7050 0    60   ~ 0
 ~DW_RST
+Text Label 6400 3050 0    60   ~ 0
+DW_XTAL1
+Text Label 2150 5700 1    60   ~ 0
+DW_XTAL1
+Text Label 9050 3550 0    60   ~ 0
+DW_SYNC
+Text Label 3950 7550 0    60   ~ 0
+DW_SYNC
 $EndSCHEMATC

Commit message: rename to tripoint...woah
Other:
- note added: "1.1"
- note added: "TriPoint"
- note added: "UWB Ranging Module"
Changed lines of the file:
@@
 LIBS:memory
 LIBS:xilinx
-LIBS:special
 LIBS:microcontrollers
 LIBS:dsp
@@
 Text Label 3950 7550 0    60   ~ 0
 DW_SYNC
+Text Notes 7400 7000 0    197  ~ 39
+TriPoint
+Text Notes 10550 7650 0    60   ~ 0
+1.1
+Text Notes 8800 7000 0    118  ~ 0
+UWB Ranging Module
 $EndSCHEMATC
