File: pcb/tritag/rev_b/tritag.brd (EAGLE design)
At the start: 46.2 x 40 mm, 47 parts, among them J1 TC2030-JLINK-NL, J2 TC2030-JLINK-NL, J3 MICRO_USB_B_HIROSE_ZX62-B-5PA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, J4 BAT_HOLE, J5 BAT_HOLE, U1 NRF51822QF, U2 TRIPOINT, U3 LTC4065, U4 MAX8887EZK33+T, X1 EPSON-FA-128

Commit message: update charging resistor on tritag
Parts:
- R3: value 2k 1% -> 560 1%
Changed lines of the file:
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@@
 <attribute name="VALUE" x="7.312828125" y="-0.489725" size="1.016" layer="28" font="vector" ratio="12" rot="MR30" align="bottom-center"/>
 </element>
-<element name="R3" library="passives" package="0402_RES" value="2k 1%" x="6.6124625" y="0.94685625" smashed="yes" rot="MR120">
+<element name="R3" library="passives" package="0402_RES" value="560 1%" x="6.6124625" y="0.94685625" smashed="yes" rot="MR120">
 <attribute name="NAME" x="6.2312125" y="0.2991625" size="1.016" layer="26" font="vector" ratio="12" rot="MR120" align="center-right"/>
 <attribute name="VALUE" x="5.40263125" y="1.645359375" size="1.016" layer="28" font="vector" ratio="12" rot="MR120" align="bottom-center"/>
