File: pcb/tritag/rev_b/tritag.sch (EAGLE design)
At the start: 47 parts, among them J1 TC2030-JLINK-NL, J2 TC2030-JLINK-NL, J3 MICRO_USB_B_HIROSE_ZX62-B-5PA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, J4 BAT_HOLE, J5 BAT_HOLE, U1 NRF51822QF, U2 TRIPOINT, U3 LTC4065, U4 MAX8887EZK33+T, X1 EPSON-FA-128

Commit message: updated tripoint module in eagle
Other:
- note added: "Must be a stable LDO for the DW1000."
Changed lines of the file:
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@@
 <plain>
 <text x="124.46" y="137.16" size="3.81" layer="98" align="bottom-center">Power Supply and Charging</text>
+<text x="201.422" y="92.71" size="1.778" layer="98" align="bottom-center">Must be a stable LDO
+for the DW1000.</text>
 </plain>
 <instances>
@@
 </schematic>
 </drawing>
+<compatibility>
+<note version="6.3" minversion="6.2.2" severity="warning">
+Since Version 6.2.2 text objects can contain more than one line,
+which will not be processed correctly with this version.
+</note>
+</compatibility>
 </eagle>

Commit message: update charging resistor on tritag
Parts:
- R3: value 2k 1% -> 560 1%
Changed lines of the file:
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@@
 <part name="R2" library="passives" deviceset="RESISTOR" device="0402_RES" value="1k"/>
 <part name="C13" library="passives" deviceset="CAPACITOR" device="" value="1uF"/>
-<part name="R3" library="passives" deviceset="RESISTOR" device="0402_RES" value="2k 1%"/>
+<part name="R3" library="passives" deviceset="RESISTOR" device="0402_RES" value="560 1%"/>
 <part name="SUPPLY5" library="supply1" deviceset="GND" device=""/>
 <part name="SUPPLY6" library="supply1" deviceset="GND" device=""/>
