File: pcb/tridev/rev_a/tridev.sch (EAGLE design)
At the start: 41 parts, among them J15 MICRO_USB_B_HIROSE_ZX62R-B-5P, J3 TC2030-JLINK-L, J4 TC2030-JLINK-L, U1 NRF51822QF, U2 TRIPOINT, U4 MAX8887EZK33+T, X1 EPSON-FA-128

Commit message: updated breakout
Parts:
- U2: value TRIPOINT -> TRIPOINT-BREAKOUT; device tripoint:TRIPOINT -> tripoint:TRIPOINT-BREAKOUT
Changed lines of the file:
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@@
 <part name="D2" library="SparkFun-LED" deviceset="LED" device="0603" value="BLUE"/>
 <part name="P+5" library="supply1" deviceset="VCC" device=""/>
-<part name="U2" library="tripoint" deviceset="TRIPOINT" device=""/>
 <part name="P+6" library="supply1" deviceset="VCC" device=""/>
 <part name="GND1" library="supply1" deviceset="GND" device=""/>
@@
 <part name="H8" library="holes" deviceset="MOUNT-HOLE" device="3.2"/>
 <part name="JP1" library="pinhead" deviceset="PINHD-2X10" device=""/>
+<part name="U2" library="tripoint" deviceset="TRIPOINT" device="-BREAKOUT"/>
 </parts>
 <sheets>
@@
 <instance part="D2" gate="G$1" x="99.06" y="111.76"/>
 <instance part="P+5" gate="VCC" x="99.06" y="132.08"/>
-<instance part="U2" gate="G$1" x="167.64" y="121.92"/>
 <instance part="P+6" gate="VCC" x="241.3" y="119.38"/>
 <instance part="GND1" gate="1" x="241.3" y="96.52"/>
@@
 <instance part="H8" gate="G$1" x="185.42" y="25.4"/>
 <instance part="JP1" gate="A" x="218.44" y="66.04"/>
+<instance part="U2" gate="G$1" x="167.64" y="121.92"/>
 </instances>
 <busses>
@@
 </segment>
 <segment>
-<pinref part="U2" gate="G$1" pin="GND"/>
 <wire x1="144.78" y1="104.14" x2="142.24" y2="104.14" width="0.1524" layer="91"/>
 <pinref part="GND2" gate="1" pin="GND"/>
 <wire x1="142.24" y1="104.14" x2="142.24" y2="96.52" width="0.1524" layer="91"/>
+<pinref part="U2" gate="G$1" pin="GND"/>
 </segment>
 <segment>
@@
 </segment>
 <segment>
-<pinref part="U2" gate="G$1" pin="VCC"/>
 <pinref part="P+7" gate="VCC" pin="VCC"/>
 <wire x1="144.78" y1="137.16" x2="142.24" y2="137.16" width="0.1524" layer="91"/>
 <wire x1="142.24" y1="137.16" x2="142.24" y2="142.24" width="0.1524" layer="91"/>
+<pinref part="U2" gate="G$1" pin="VCC"/>
 </segment>
 </net>
@@
 <net name="DW_INT" class="0">
 <segment>
-<pinref part="U2" gate="G$1" pin="INTERRUPT"/>
 <wire x1="144.78" y1="124.46" x2="111.76" y2="124.46" width="0.1524" layer="91"/>
 <wire x1="111.76" y1="124.46" x2="111.76" y2="93.98" width="0.1524" layer="91"/>
@@
 <wire x1="91.44" y1="93.98" x2="91.44" y2="81.28" width="0.1524" layer="91"/>
 <junction x="91.44" y="81.28"/>
+<pinref part="U2" gate="G$1" pin="INTERRUPT"/>
 </segment>
 </net>
@@
 <wire x1="86.36" y1="71.12" x2="109.22" y2="71.12" width="0.1524" layer="91"/>
 <wire x1="109.22" y1="71.12" x2="109.22" y2="129.54" width="0.1524" layer="91"/>
-<pinref part="U2" gate="G$1" pin="SDA"/>
 <wire x1="109.22" y1="129.54" x2="119.38" y2="129.54" width="0.1524" layer="91"/>
 <wire x1="119.38" y1="129.54" x2="144.78" y2="129.54" width="0.1524" layer="91"/>
@@
 <junction x="119.38" y="137.16"/>
 <junction x="119.38" y="129.54"/>
+<pinref part="U2" gate="G$1" pin="SDA"/>
 </segment>
 </net>
@@
 <wire x1="127" y1="137.16" x2="129.54" y2="137.16" width="0.1524" layer="91"/>
 <label x="129.54" y="137.16" size="1.27" layer="95" xref="yes"/>
-<pinref part="U2" gate="G$1" pin="SCL"/>
 <wire x1="144.78" y1="132.08" x2="127" y2="132.08" width="0.1524" layer="91"/>
 <wire x1="127" y1="132.08" x2="106.68" y2="132.08" width="0.1524" layer="91"/>
@@
 <junction x="127" y="137.16"/>
 <junction x="127" y="132.08"/>
+<pinref part="U2" gate="G$1" pin="SCL"/>
 </segment>
 </net>
@@
 <net name="N$1" class="0">
 <segment>
-<pinref part="U2" gate="G$1" pin="ANT1"/>
 <wire x1="187.96" y1="134.62" x2="195.58" y2="134.62" width="0.1524" layer="91"/>
 <wire x1="195.58" y1="134.62" x2="195.58" y2="144.78" width="0.1524" layer="91"/>
+<pinref part="U2" gate="G$1" pin="ANT1"/>
 </segment>
 </net>
 <net name="N$2" class="0">
 <segment>
-<pinref part="U2" gate="G$1" pin="ANT2"/>
 <wire x1="187.96" y1="129.54" x2="213.36" y2="129.54" width="0.1524" layer="91"/>
 <wire x1="213.36" y1="129.54" x2="213.36" y2="144.78" width="0.1524" layer="91"/>
+<pinref part="U2" gate="G$1" pin="ANT2"/>
 </segment>
 </net>
 <net name="N$3" class="0">
 <segment>
-<pinref part="U2" gate="G$1" pin="ANT3"/>
 <wire x1="187.96" y1="124.46" x2="231.14" y2="124.46" width="0.1524" layer="91"/>
 <wire x1="231.14" y1="124.46" x2="231.14" y2="144.78" width="0.1524" layer="91"/>
+<pinref part="U2" gate="G$1" pin="ANT3"/>
 </segment>
 </net>
 <net name="N$4" class="0">
 <segment>
-<pinref part="U2" gate="G$1" pin="SWDIO"/>
 <wire x1="187.96" y1="111.76" x2="195.58" y2="111.76" width="0.1524" layer="91"/>
 <wire x1="195.58" y1="111.76" x2="195.58" y2="114.3" width="0.1524" layer="91"/>
 <wire x1="195.58" y1="114.3" x2="213.36" y2="114.3" width="0.1524" layer="91"/>
 <pinref part="J3" gate="G$1" pin="SWDIO"/>
+<pinref part="U2" gate="G$1" pin="SWDIO"/>
 </segment>
 </net>
@@
 <wire x1="213.36" y1="111.76" x2="198.12" y2="111.76" width="0.1524" layer="91"/>
 <wire x1="198.12" y1="111.76" x2="198.12" y2="109.22" width="0.1524" layer="91"/>
-<pinref part="U2" gate="G$1" pin="SWDCLK"/>
 <wire x1="198.12" y1="109.22" x2="187.96" y2="109.22" width="0.1524" layer="91"/>
 <pinref part="J3" gate="G$1" pin="SWDCLK"/>
+<pinref part="U2" gate="G$1" pin="SWDCLK"/>
 </segment>
 </net>
 <net name="N$8" class="0">
 <segment>
-<pinref part="U2" gate="G$1" pin="!RESET"/>
 <wire x1="187.96" y1="106.68" x2="198.12" y2="106.68" width="0.1524" layer="91"/>
 <wire x1="198.12" y1="106.68" x2="198.12" y2="104.14" width="0.1524" layer="91"/>
 <wire x1="198.12" y1="104.14" x2="213.36" y2="104.14" width="0.1524" layer="91"/>
 <pinref part="J3" gate="G$1" pin="!RESET"/>
-</segment>
-</net>
+<pinref part="U2" gate="G$1" pin="!RESET"/>
+</segment>
+</net>

Commit message: breakout basically done
Parts:
- removed J15: MICRO_USB_B_HIROSE_ZX62R-B-5P, connector:MICRO_USB_B_HIROSE_ZX62R-B-5P
- added C16, C17, C18, C19, C20, C22, C24, C25, C9: 0.1uF, passives:CAPACITOR
- added C21, C23: 4.7uF, passives:CAP_POL0603
- added C26, C27: 18pF, passives:CAPACITOR
- added D3: RED, SparkFun-LED:LED0603
- added D4: BLUE, SparkFun-LED:LED0603
- added J1: MICRO_USB_B_HIROSE_ZX62R-B-5P, connector:MICRO_USB_B_HIROSE_ZX62R-B-5P
- added J5, J6: (no value), SparkFun-Passives:JUMPER-2PTH
- added L3, L4, L5: FERRITE_BEAD, passives:FERRITE_BEAD
- added R3: 12k 1%, passives:RESISTOR0402_RES
- added R7, R8: 1k, passives:RESISTOR0402_RES
- added U5: FT232HQ, chips:FT232HQ
- added X2: TXC-8Z-12MHZ, crystals:TXC-8Z-12MHZ
- renumbered H5 to H1, H6 to H2, H7 to H3, H8 to H4, JP1 to J2
Connections:
- removed net DW_INT: U1.P25, U2.INTERRUPT
- new net !DW_CS: J2.5, U2.!DEBUG_DW_CS
- new net !DW_RST: J2.6, U2.!DEBUG_DW_RST
- new net DW_CLK: J2.4, U2.DEBUG_DW_CLK
- new net DW_IRQ: J2.15, U2.DEBUG_DW_IRQ
- new net DW_MISO: J2.3, U2.DEBUG_DW_MISO
- new net DW_MOSI: J2.2, U2.DEBUG_DW_MOSI
- new net DW_SYNC: J2.1, U2.DW_SYNC
- new net DW_XTAL1: J2.16, U2.DW_XTAL1
- new net N$12: C20.1, C21.CATHODE, L5.P$2, U5.VREGIN
- new net N$13: C24.1, U5.VCCCORE
- new net N$14: C26.1, U5.XCS0, X2.2
- new net N$16: C27.1, U5.XCS1, X2.1
- new net N$21: C25.1, U5.VCCA
- new net N$22: R3.2, U5.REF
- new net N$23: J5.2, U2.VCC
- new net N$24: D3.A, R7.1
- new net N$25: D4.A, R8.1
- new net N$26: D4.C, U5.ADBUS4
- new net N$38: J2.17
- new net N$5: D3.C, U5.ADBUS3
- new net NRF_VCC: C14.1, C8.1, J4.VCC, J6.2, R1.2, U1.VDD
- new net TP_GPIO0: J2.7, U2.GPIO0
- new net TP_GPIO1: J2.8, U2.GPIO1
- new net TP_GPIO2: J2.9, U2.GPIO2
- new net TP_GPIO3: J2.10, U2.GPIO3
- new net TP_GPIO4: J2.11, U2.GPIO4
- new net TP_INT: J2.14, U1.P25, U2.INTERRUPT
- new net USB_D+: J1.D+, U5.DP
- new net USB_D-: J1.D-, U5.DM
- new net VCC3V3: C16.1, C17.1, C22.1, C23.CATHODE, C9.1, L3.P$2, L4.P$2, R7.2, R8.2, U5.!RESET, U5.VCCD, U5.VCCIO
- new net VPHY: C19.1, L3.P$1, U5.VPHY
- new net VPLL: C18.1, L4.P$1, U5.VPLL
- net GND: now also C16.2, C17.2, C18.2, C19.2, C20.2, C21.ANODE, C22.2, C23.ANODE, C24.2, C25.2, C26.2, C27.2, C9.2, J1.GND, J2.19, J2.20, R3.1, U5.GND, U5.TEST, X2.GND; no longer J15.GND
- net I2C_SCL: now also J2.13, U5.ADBUS0
- net I2C_SDA: now also J2.12, U5.ADBUS1, U5.ADBUS2
- net N$1: now also A1.ANT
- net N$2: now also A2.ANT
- net N$3: now also A3.ANT
- net VCC: now also J2.18, J5.1, J6.1; no longer C14.1, C8.1, J4.VCC, R1.2, U1.VDD, U2.VCC
- net VUSB: now also J1.+5V, L5.P$1; no longer J15.+5V
Other:
- note added: "I2C over USB Interface"
- note added: "PIN12"
- note added: "PIN24"
- note added: "PIN46"
- note added: "TriPoint Power Supply"
- note removed: "Power Supply and Charging"
- moved on the sheet: C10, C11, C13, C15, D1, D2, R1, R2, R4, R5, U4

Commit message: updated parts, added bom
Parts:
- removed C4: 1nF, passives:CAPACITOR
- removed C5: 2.2nF, passives:CAPACITOR
- removed U5: FT232HQ, chips:FT232HQ
- added C44, C55: 18pF, passives:CAPACITOR
- added U3: MAX8887EZK33+T, chips:MAX8887EZK33+T
- C10, C11, C14: value 4.7uF -> 0.1uF
- C12, C13: value 1uF -> 0.1uF
- C15: value 10nF -> 0.1uF
- C21: value 4.7uF -> 1uF; device passives:CAP_POL0603 -> passives:CAPACITOR; DIGIKEY 478-8656-1-ND -> (none)
- C22: value 0.1uF -> 1uF
- C23: device passives:CAP_POL0603 -> passives:CAPACITOR; DIGIKEY 478-8656-1-ND -> (none)
- C24, C25: value 0.1uF -> 4.7uF
- C26, C27: value 18pF -> 4.7uF; device passives:CAPACITOR -> passives:CAP_POL0603; DIGIKEY (none) -> 478-8656-1-ND
- C6: value 47nF -> 1nF
- C7: value 0.1uF -> 2.2nF
- C8: value 0.1uF -> 10nF
- C9: value 0.1uF -> 47nF
- D3: value RED -> BLUE
- D4: value BLUE -> RED
- J3, J4: value TC2030-JLINK-L -> (none); device connector:TC2030-JLINK-L -> SparkFun-Passives:JUMPER-2PTH
- J5, J6: value (none) -> TC2030-JLINK-L; device SparkFun-Passives:JUMPER-2PTH -> connector:TC2030-JLINK-L
- R3: value 12k 1% -> 1k
- R4: value 10k -> 1k
- R6: value 12k -> 10k
- R7: value 1k -> 12k
- R8: value 1k -> 12k 1%
- U1: value NRF51822QF -> TRIPOINT-BREAKOUT; device chips:NRF51822QF -> tripoint:TRIPOINT-BREAKOUT
- U2: value TRIPOINT-BREAKOUT -> NRF51822QF; device tripoint:TRIPOINT-BREAKOUT -> chips:NRF51822QF
- U4: value MAX8887EZK33+T -> FT232HQ; device chips:MAX8887EZK33+T -> chips:FT232HQ
Connections:
- net !DW_CS: now also U1.!DEBUG_DW_CS; no longer U2.!DEBUG_DW_CS
- net !DW_RST: now also U1.!DEBUG_DW_RST; no longer U2.!DEBUG_DW_RST
- net AVDD: now also C21.1, C6.1, U2.AVDD; no longer C12.1, C4.1, U1.AVDD
- net BATIN: now also U2.P01/AIN2; no longer U1.P01/AIN2
- net DCC: now also U2.DCC; no longer U1.DCC
- net DW_CLK: now also U1.DEBUG_DW_CLK; no longer U2.DEBUG_DW_CLK
- net DW_IRQ: now also U1.DEBUG_DW_IRQ; no longer U2.DEBUG_DW_IRQ
- net DW_MISO: now also U1.DEBUG_DW_MISO; no longer U2.DEBUG_DW_MISO
- net DW_MOSI: now also U1.DEBUG_DW_MOSI; no longer U2.DEBUG_DW_MOSI
- net DW_SYNC: now also U1.DW_SYNC; no longer U2.DW_SYNC
- net DW_XTAL1: now also U1.DW_XTAL1; no longer U2.DW_XTAL1
- net GND: now also C21.2, C23.2, C26.ANODE, C27.ANODE, C44.2, C55.2, J5.GND, J6.GND, R7.1, R8.1, U3.GND, U4.TEST; no longer C21.ANODE, C23.ANODE, C26.2, C27.2, C4.2, C5.2, J3.GND, J4.GND, R3.1, R6.1, U5.GND, U5.TEST
- net I2C_SCL: now also U1.SCL, U2.P28, U4.ADBUS0; no longer U1.P28, U2.SCL, U5.ADBUS0
- net I2C_SDA: now also R6.1, U1.SDA, U2.P29, U4.ADBUS1, U4.ADBUS2; no longer R4.1, U1.P29, U2.SDA, U5.ADBUS1, U5.ADBUS2
- net N$1: now also U1.ANT1; no longer U2.ANT1
- net N$10: now also U2.XC2; no longer U1.XC2
- net N$11: now also C8.1, U3.BP; no longer C15.1, U4.BP
- net N$12: now also C26.CATHODE, U4.VREGIN; no longer C21.CATHODE, U5.VREGIN
- net N$13: now also C14.1, U4.VCCCORE; no longer C24.1, U5.VCCCORE
- net N$14: now also C55.1, U4.XCS0; no longer C26.1, U5.XCS0
- net N$15: now also C9.1, U2.DEC2; no longer C6.1, U1.DEC2
- net N$16: now also C44.1, U4.XCS1; no longer C27.1, U5.XCS1
- net N$17: now also C10.1, U2.DEC1; no longer C7.1, U1.DEC1
- net N$18: now also U2.ANT1; no longer U1.ANT1
- net N$19: now also U2.ANT2; no longer U1.ANT2
- net N$2: now also U1.ANT2; no longer U2.ANT2
- net N$20: now also C7.1, U2.VDD_PA; no longer C5.1, U1.VDD_PA
- net N$21: now also C15.1, U4.VCCA; no longer C25.1, U5.VCCA
- net N$22: now also R8.2, U4.REF; no longer R3.2, U5.REF
- net N$23: now also J4.2, U1.VCC; no longer J5.2, U2.VCC
- net N$24: now also D4.A, R3.1; no longer D3.A, R7.1
- net N$25: now also D3.A, R4.1; no longer D4.A, R8.1
- net N$26: now also D3.C, U4.ADBUS4; no longer D4.C, U5.ADBUS4
- net N$3: now also U1.ANT3; no longer U2.ANT3
- net N$4: now also J5.SWDIO, U1.SWDIO; no longer J3.SWDIO, U2.SWDIO
- net N$5: now also D4.C, U4.ADBUS3; no longer D3.C, U5.ADBUS3
- net N$6: now also U2.P17; no longer U1.P17
- net N$7: now also J5.SWDCLK, U1.SWDCLK; no longer J3.SWDCLK, U2.SWDCLK
- net N$8: now also J5.!RESET, U1.!RESET; no longer J3.!RESET, U2.!RESET
- net N$9: now also U2.XC1; no longer U1.XC1
- net NRF_VCC: now also C11.1, C25.1, J3.2, J6.VCC, U2.VDD; no longer C14.1, C8.1, J4.VCC, J6.2, U1.VDD
- net SWDCLK: now also J6.SWDCLK, R7.2, U2.SWDCLK; no longer J4.SWDCLK, R6.2, U1.SWDCLK
- net SWDIO/!RESET: now also J6.SWDIO, U2.SWDIO/!RESET; no longer J4.SWDIO, U1.SWDIO/!RESET
- net TP_GPIO0: now also U1.GPIO0; no longer U2.GPIO0
- net TP_GPIO1: now also U1.GPIO1; no longer U2.GPIO1
- net TP_GPIO2: now also U1.GPIO2; no longer U2.GPIO2
- net TP_GPIO3: now also U1.GPIO3; no longer U2.GPIO3
- net TP_GPIO4: now also U1.GPIO4; no longer U2.GPIO4
- net TP_INT: now also U1.INTERRUPT, U2.P25; no longer U1.P25, U2.INTERRUPT
- net USB_D+: now also U4.DP; no longer U5.DP
- net USB_D-: now also U4.DM; no longer U5.DM
- net VCC: now also C24.1, J3.1, J4.1, J5.VCC, R6.2, U3.OUT; no longer C11.1, J3.VCC, J5.1, J6.1, R4.2, U4.OUT
- net VCC3V3: now also C12.1, C13.1, C27.CATHODE, R3.2, R4.2, U4.!RESET, U4.VCCD, U4.VCCIO; no longer C22.1, C23.CATHODE, C9.1, R7.2, R8.2, U5.!RESET, U5.VCCD, U5.VCCIO
- net VPHY: now also U4.VPHY; no longer U5.VPHY
- net VPLL: now also U4.VPLL; no longer U5.VPLL
- net VUSB: now also C22.1, C23.1, U3.!SHDN, U3.IN; no longer C10.1, C13.1, U4.!SHDN, U4.IN
Other:
- moved on the sheet: C13, C15, C22, C24, C6, C7, D3, D4, R3, R6, R8
