File: pcb/calibration-brace/calibration-brace.kicad_pcb (KiCad board)
At the start: 2 copper layers, 5 x 44.1 mm, 21 parts, among them U1 120220-0315, U10 120220-0315, U11 120220-0315, U12 120220-0315, U13 120220-0315, U14 120220-0315, U15 120220-0315, U16 120220-0315, U17 120220-0315, U18 BRACE-CASTELLATION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

Commit message: done editing brace
Parts:
- added U22: 120220-0315, polypoint:120220-0315, B.Cu at (152.4, 109.5)
- added U23: 120220-0315, polypoint:120220-0315, B.Cu at (152.4, 103.2)
- added U24: 120220-0315, polypoint:120220-0315, B.Cu at (152.4, 104.8)
- added U25: 120220-0315, polypoint:120220-0315, B.Cu at (152.4, 111.1)
- added U26: 120220-0315, polypoint:120220-0315, B.Cu at (152.4, 106.4)
- added U27: 120220-0315, polypoint:120220-0315, B.Cu at (152.4, 108.0)
- added U28: 120220-0315, polypoint:120220-0315, B.Cu at (152.4, 115.9)
- added U29: 120220-0315, polypoint:120220-0315, B.Cu at (152.4, 112.7)
- added U30: 120220-0315, polypoint:120220-0315, B.Cu at (152.4, 123.8)
- added U31: 120220-0315, polypoint:120220-0315, B.Cu at (152.4, 101.6)
- added U32: 120220-0315, polypoint:120220-0315, B.Cu at (152.4, 117.5)
- added U33: 120220-0315, polypoint:120220-0315, B.Cu at (152.4, 120.7)
- added U34: 120220-0315, polypoint:120220-0315, B.Cu at (152.4, 114.3)
- added U35: 120220-0315, polypoint:120220-0315, B.Cu at (152.4, 119.1)
- added U36: 120220-0315, polypoint:120220-0315, B.Cu at (152.4, 125.4)
- added U37: 120220-0315, polypoint:120220-0315, B.Cu at (152.4, 127.0)
- added U38: 120220-0315, polypoint:120220-0315, B.Cu at (152.4, 122.2)
- U18, U21: value BRACE-CASTELLATION -> 120220-0315; footprint polypoint:BRACE-CASTELLATION -> polypoint:120220-0315
- U19, U20: value BRACE-CASTELLATION -> 120220-0315; footprint polypoint:BRACE-CASTELLATION -> polypoint:120220-0315; moved to B.Cu
- moved U20 4.76 mm to (152.4, 130.8)
- moved U21 4.76 mm to (152.4, 97.8)
- moved U19 2.53 mm to (152.4, 97.8)
- moved U18 2.53 mm to (152.4, 130.8)
Connections:
- U18 pad 1: Net-(U18-Pad1) -> (no net)
- U19 pad 1: Net-(U19-Pad1) -> (no net)
- U20 pad 1: Net-(U20-Pad1) -> (no net)
- U21 pad 1: Net-(U21-Pad1) -> (no net)
Routing:
- net Net-(U29-Pad1): track 0.00 -> 2.41 mm, vias 0 -> 3
- net Net-(U28-Pad1): track 0.00 -> 2.41 mm, vias 0 -> 3
- net Net-(U13-Pad1): track 0.00 -> 1.20 mm, vias 0 -> 3
- net Net-(U30-Pad1): vias 0 -> 1
- net Net-(U27-Pad1): vias 0 -> 1
- net Net-(U26-Pad1): vias 0 -> 1
- net Net-(U25-Pad1): vias 0 -> 1
- net Net-(U24-Pad1): vias 0 -> 1
- net Net-(U2-Pad1): vias 0 -> 1
- net Net-(U17-Pad1): vias 0 -> 1
- net Net-(U16-Pad1): vias 0 -> 1
- net Net-(U15-Pad1): vias 0 -> 1
- net Net-(U14-Pad1): vias 0 -> 1
- net Net-(U12-Pad1): vias 0 -> 1
- net Net-(U11-Pad1): vias 0 -> 1
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Other:
- board size 5 x 44.1 mm -> 4.9 x 38.1 mm
