File: pcb/calibration-brace/calibration-brace.sch (KiCad schematic (older format))
At the start: 21 parts, among them U1 120220-0315, U10 120220-0315, U11 120220-0315, U12 120220-0315, U13 120220-0315, U14 120220-0315, U15 120220-0315, U16 120220-0315, U17 120220-0315, U18 BRACE-CASTELLATION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

Commit message: done editing brace
Parts:
- removed U18, U19, U20, U21: BRACE-CASTELLATION, polypoint:BRACE-CASTELLATION, symbol BRACE-CASTELLATION
- added U18, U19, U20, U21, U22, U23, U24, U25, U26, U27, U28, U29, U30, U31, U32, U33, U34, U35, U36, U37, U38: 120220-0315, polypoint:120220-0315, symbol 120220-0315
Connections:
- net at U1.1: now also U22.1
- net at U2.1: now also U23.1
- net at U3.1: now also U24.1
- net at U4.1: now also U25.1
- net at U5.1: now also U26.1
- net at U6.1: now also U27.1
- net at U7.1: now also U28.1
- net at U8.1: now also U29.1
- net at U9.1: now also U30.1
- net at U10.1: now also U31.1
- net at U11.1: now also U32.1
- net at U12.1: now also U33.1
- net at U13.1: now also U34.1
- net at U14.1: now also U35.1
- net at U15.1: now also U36.1
- net at U16.1: now also U37.1
- net at U17.1: now also U38.1
