File: pcb/pinpoint/pinpoint_tridev_adapter/pinpoint_tridev_adapter.kicad_pcb (KiCad board)
At the start: 4 copper layers, 27.9 x 50.8 mm, 27 parts, among them J1 RJ45, P1 SMA, P2 CONN_01X03, P3 SMA, P4 CONN_01X06, P5 CONN_01X03, P6 CONN_02X10, P7 CONN_01X02, U1 AOZ1282CI, U2 MAX8877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

Commit message: adding component part numbers
Changed lines of the file:
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@@
     (links 66)
     (no_connects 0)
-    (area 104.064999 46.914999 132.155001 97.865001)
+    (area 101.670067 43.7823 132.510601 99.1966)
     (thickness 1.6)
-    (drawings 12)
+    (drawings 13)
     (tracks 207)
     (zones 0)
@@
   )
   (setup
-    (last_trace_width 1.27)
+    (last_trace_width 0.1016)
     (user_trace_width 0.1016)
     (user_trace_width 0.254)
@@
     )
   )
+  (gr_text GND (at 109.601 67.31) (layer F.SilkS)
+    (effects (font (size 0.762 0.762) (thickness 0.1905)))
+  )
   (gr_text "PinPoint to\nTriDev Adapter\nv0.1\nBen Kempke" (at 104.775 81.407) (layer F.SilkS)

Commit message: minor cosmetic fixes
Other:
- copper layers 4 -> 2
Changed lines of the file:
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@@
     (links 66)
     (no_connects 0)
-    (area 101.670067 43.7823 132.510601 99.1966)
+    (area 104.064999 46.914999 132.155001 97.865001)
     (thickness 1.6)
     (drawings 13)
@@
   (layers
     (0 F.Cu signal)
-    (1 In1.Cu signal)
-    (2 In2.Cu signal)
     (31 B.Cu signal)
     (32 B.Adhes user)
