File: pcb/pinpoint/pinpoint_tridev_adapter/pinpoint_tridev_adapter.sch (KiCad schematic (older format))
At the start: 27 parts, among them J1 RJ45, P1 SMA, P2 CONN_01X03, P3 SMA, P4 CONN_01X06, P5 CONN_01X03, P6 CONN_02X10, P7 CONN_01X02, U1 AOZ1282CI, U2 MAX8877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

Commit message: adding component part numbers
Parts:
- C1: value C_Small -> 0.1uF; DistPartNo (none) -> 490-10458-1-ND; ManPartNo (none) -> GRM155R62A104KE14D
- C2, C3: DistPartNo (none) -> 490-10751-1-ND; ManPartNo (none) -> GRM21BR61H475KE51L
- C4: DistPartNo (none) -> 490-6473-1-ND; ManPartNo (none) -> GRM21BR61C106KE15K
- C5: DistPartNo (none) -> 490-4516-1-ND; ManPartNo (none) -> GRM155R71H103KA88D
- C6, C7, C8: DistPartNo (none) -> 490-10458-1-ND; ManPartNo (none) -> GRM155R62A104KE14D
- J1: DistPartNo (none) -> AE10387-ND; ManPartNo (none) -> A-2004-2-4-LPS-N-R
- L1: value INDUCTOR_SMALL -> 22uH; DistPartNo (none) -> 587-2082-1-ND; ManPartNo (none) -> NR6045T220M
- P1, P3: DistPartNo (none) -> CONSMA003.062-ND; ManPartNo (none) -> CONSMA003.062
- P6: DistPartNo (none) -> SAM1204-10-ND; ManPartNo (none) -> SSQ-110-03-T-D
- R1: DistPartNo (none) -> P4.70KLCT-ND; ManPartNo (none) -> ERJ-2RKF4701X
- R2, R5: DistPartNo (none) -> P100LCT-ND; ManPartNo (none) -> ERJ-2RKF1000X
- R3: DistPartNo (none) -> P49.9KLCT-ND; ManPartNo (none) -> ERJ-2RKF4992X
- R4: DistPartNo (none) -> P9.53KLCT-ND; ManPartNo (none) -> ERJ-2RKF9531X
- U1: DistPartNo (none) -> 785-1613-1-ND; ManPartNo (none) -> AOZ1282CI
- U2: DistPartNo (none) -> MAX8877EUK33+CT-ND; ManPartNo (none) -> MAX8877EUK33+T
- U3, U4: DistPartNo (none) -> 800-3330-5-ND; ManPartNo (none) -> 830S21AMI-01LF
Changed lines of the file:
@@
 F 2 "Pin_Headers:Pin_Header_Straight_2x10" H 6000 3550 60  0001 C CNN
 F 3 "" H 6000 3550 60  0000 C CNN
+F 4 "SSQ-110-03-T-D" H 6000 4750 60  0001 C CNN "ManPartNo"
+F 5 "SAM1204-10-ND" H 6000 4750 60  0001 C CNN "DistPartNo"
 	1    6000 4750
 	1    0    0    -1
@@
 F 2 "polypoint:RJ45_8" H 9250 1700 60  0001 C CNN
 F 3 "" H 9250 1700 60  0000 C CNN
+F 4 "A-2004-2-4-LPS-N-R" V 9250 1700 60  0001 C CNN "ManPartNo"
+F 5 "AE10387-ND" V 9250 1700 60  0001 C CNN "DistPartNo"
 	1    9250 1700
 	0    1    1    0
@@
 F 2 "TO_SOT_Packages_SMD:SOT-23-6" H 3600 1600 60  0001 C CNN
 F 3 "" H 3600 1600 60  0000 C CNN
+F 4 "AOZ1282CI" H 3600 1600 60  0001 C CNN "ManPartNo"
+F 5 "785-1613-1-ND" H 3600 1600 60  0001 C CNN "DistPartNo"
 	1    3600 1600
 	1    0    0    -1
@@
 F 2 "Resistors_SMD:R_0402" H 8300 1450 60  0001 C CNN
 F 3 "" H 8300 1450 60  0000 C CNN
+F 4 " ERJ-2RKF1000X" V 8300 1450 60  0001 C CNN "ManPartNo"
+F 5 "P100LCT-ND" V 8300 1450 60  0001 C CNN "DistPartNo"
 	1    8300 1450
 	0    1    1    0
@@
 F 2 "Resistors_SMD:R_0402" H 8300 2050 60  0001 C CNN
 F 3 "" H 8300 2050 60  0000 C CNN
+F 4 "ERJ-2RKF1000X" V 8300 2050 60  0001 C CNN "ManPartNo"
+F 5 "P100LCT-ND" V 8300 2050 60  0001 C CNN "DistPartNo"
 	1    8300 2050
 	0    1    1    0
@@
 F 2 "Resistors_SMD:R_0402" H 2950 1200 60  0001 C CNN
 F 3 "" H 2950 1200 60  0000 C CNN
+F 4 "ERJ-2RKF4701X" H 2950 1200 60  0001 C CNN "ManPartNo"
+F 5 "P4.70KLCT-ND" H 2950 1200 60  0001 C CNN "DistPartNo"
 	1    2950 1200
 	1    0    0    -1
@@
 F 2 "Capacitors_SMD:C_0805" H 2300 1200 60  0001 C CNN
 F 3 "" H 2300 1200 60  0000 C CNN
+F 4 "GRM21BR61H475KE51L" H 2300 1200 60  0001 C CNN "ManPartNo"
+F 5 "490-10751-1-ND" H 2300 1200 60  0001 C CNN "DistPartNo"
 	1    2300 1200
 	1    0    0    -1
@@
 P 4100 1050
 F 0 "C1" V 3870 1050 50  0000 C CNN
-F 1 "C_Small" V 3962 1050 50  0000 C CNN
+F 1 "0.1uF" V 3962 1050 50  0000 C CNN
 F 2 "Capacitors_SMD:C_0402" H 4100 1050 60  0001 C CNN
 F 3 "" H 4100 1050 60  0000 C CNN
+F 4 "GRM155R62A104KE14D" V 4100 1050 60  0001 C CNN "ManPartNo"
+F 5 "490-10458-1-ND" V 4100 1050 60  0001 C CNN "DistPartNo"
 	1    4100 1050
 	0    1    1    0
@@
 F 2 "Resistors_SMD:R_0402" H 5200 1650 60  0001 C CNN
 F 3 "" H 5200 1650 60  0000 C CNN
+F 4 "ERJ-2RKF4992X" H 5200 1650 60  0001 C CNN "ManPartNo"
+F 5 "P49.9KLCT-ND" H 5200 1650 60  0001 C CNN "DistPartNo"
 	1    5200 1650
 	1    0    0    -1
@@
 F 2 "Resistors_SMD:R_0402" H 5200 1950 60  0001 C CNN
 F 3 "" H 5200 1950 60  0000 C CNN
+F 4 "ERJ-2RKF9531X" H 5200 1950 60  0001 C CNN "ManPartNo"
+F 5 "P9.53KLCT-ND" H 5200 1950 60  0001 C CNN "DistPartNo"
 	1    5200 1950
 	1    0    0    -1
@@
 P 4850 1550
 F 0 "L1" H 4850 1766 50  0000 C CNN
-F 1 "INDUCTOR_SMALL" H 4850 1674 50  0000 C CNN
+F 1 "22uH" H 4850 1674 50  0000 C CNN
 F 2 "polypoint:NR6045" H 4850 1550 60  0001 C CNN
 F 3 "" H 4850 1550 60  0000 C CNN
+F 4 "NR6045T220M" H 4850 1550 60  0001 C CNN "ManPartNo"
+F 5 "587-2082-1-ND" H 4850 1550 60  0001 C CNN "DistPartNo"
 	1    4850 1550
 	1    0    0    -1
@@
 F 2 "TO_SOT_Packages_SMD:SOT-23-5" H 6650 1650 60  0001 C CNN
 F 3 "" H 6650 1650 60  0000 C CNN
+F 4 "MAX8877EUK33+T" H 6650 1650 60  0001 C CNN "ManPartNo"
+F 5 "MAX8877EUK33+CT-ND" H 6650 1650 60  0001 C CNN "DistPartNo"
 	1    6650 1650
 	1    0    0    -1
@@
 F 2 "Capacitors_SMD:C_0805" H 5600 1700 60  0001 C CNN
 F 3 "" H 5600 1700 60  0000 C CNN
+F 4 "GRM21BR61C106KE15K" H 5600 1700 60  0001 C CNN "ManPartNo"
+F 5 "490-6473-1-ND" H 5600 1700 60  0001 C CNN "DistPartNo"
 	1    5600 1700
 	1    0    0    -1
@@
 F 2 "Capacitors_SMD:C_0402" H 6100 1950 60  0001 C CNN
 F 3 "" H 6100 1950 60  0000 C CNN
+F 4 "GRM155R71H103KA88D" H 6100 1950 60  0001 C CNN "ManPartNo"
+F 5 "490-4516-1-ND" H 6100 1950 60  0001 C CNN "DistPartNo"
 	1    6100 1950
 	1    0    0    -1
@@
 F 2 "Capacitors_SMD:C_0805" H 7450 1650 60  0001 C CNN
 F 3 "" H 7450 1650 60  0000 C CNN
+F 4 "GRM21BR61H475KE51L" H 7450 1650 60  0001 C CNN "ManPartNo"
+F 5 "490-10751-1-ND" H 7450 1650 60  0001 C CNN "DistPartNo"
 	1    7450 1650
 	1    0    0    -1
@@
 F 2 "Housings_SOIC:SOIC-8_3.9x4.9mm_Pitch1.27mm" H 4000 3250 60  0001 C CNN
 F 3 "" H 4000 3250 60  0000 C CNN
+F 4 "830S21AMI-01LF" H 4000 3400 60  0001 C CNN "ManPartNo"
+F 5 "800-3330-5-ND" H 4000 3400 60  0001 C CNN "DistPartNo"
 	1    4000 3400
 	1    0    0    -1
@@
 F 2 "Housings_SOIC:SOIC-8_3.9x4.9mm_Pitch1.27mm" H 4000 4150 60  0001 C CNN
 F 3 "" H 4000 4150 60  0000 C CNN
+F 4 "830S21AMI-01LF" H 4000 4300 60  0001 C CNN "ManPartNo"
+F 5 "800-3330-5-ND" H 4000 4300 60  0001 C CNN "DistPartNo"
 	1    4000 4300
 	1    0    0    -1
@@
 F 2 "Capacitors_SMD:C_0402" H 3250 4150 60  0001 C CNN
 F 3 "" H 3250 4150 60  0000 C CNN
+F 4 "GRM155R62A104KE14D" V 3250 4150 60  0001 C CNN "ManPartNo"
+F 5 "490-10458-1-ND" V 3250 4150 60  0001 C CNN "DistPartNo"
 	1    3250 4150
 	0    1    1    0
@@
 F 2 "Capacitors_SMD:C_0402" H 3250 3250 60  0001 C CNN
 F 3 "" H 3250 3250 60  0000 C CNN
+F 4 "GRM155R62A104KE14D" V 3250 3250 60  0001 C CNN "ManPartNo"
+F 5 "490-10458-1-ND" V 3250 3250 60  0001 C CNN "DistPartNo"
 	1    3250 3250
 	0    1    1    0
@@
 F 2 "Capacitors_SMD:C_0402" H 5300 3200 60  0001 C CNN
 F 3 "" H 5300 3200 60  0000 C CNN
+F 4 "GRM155R62A104KE14D" V 5300 3200 60  0001 C CNN "ManPartNo"
+F 5 "490-10458-1-ND" V 5300 3200 60  0001 C CNN "DistPartNo"
 	1    5300 3200
 	0    1    1    0
@@
 F 2 "polypoint:SMA_EDGE" H 5300 4300 60  0001 C CNN
 F 3 "" H 5300 4300 60  0000 C CNN
+F 4 "CONSMA003.062" H 5300 4300 60  0001 C CNN "ManPartNo"
+F 5 "CONSMA003.062-ND" H 5300 4300 60  0001 C CNN "DistPartNo"
 	1    5300 4300
 	1    0    0    -1
@@
 F 2 "polypoint:SMA_EDGE" H 5300 3400 60  0001 C CNN
 F 3 "" H 5300 3400 60  0000 C CNN
+F 4 "CONSMA003.062" H 5300 3400 60  0001 C CNN "ManPartNo"
+F 5 "CONSMA003.062-ND" H 5300 3400 60  0001 C CNN "DistPartNo"
 	1    5300 3400
 	1    0    0    -1

Commit message: adding BOMs for two PinPoint boards
Parts:
- D1: DistPartNo (none) -> BSR106WS-TPMSCT-ND; ManPartNo (none) -> BSR106WS-TP
Changed lines of the file:
@@
 F 2 "Diodes_SMD:SOD-323" H 4500 1800 60  0001 C CNN
 F 3 "" H 4500 1800 60  0000 C CNN
+F 4 "BSR106WS-TP" V 4500 1800 60  0001 C CNN "ManPartNo"
+F 5 "BSR106WS-TPMSCT-ND" V 4500 1800 60  0001 C CNN "DistPartNo"
 	1    4500 1800
 	0    1    1    0
